Commit message: Update urdf to take into account new textures

File: urdf/pepper_1.7/pepper.urdf (robot description, URDF)
Before this commit: robot JulietteY20MP, 82 links, 81 joints
Links:
- added link HeadPitch_face_shiny; visual mesh filename=meshes/pepper_1.7/HeadPitch_face_shiny.obj scale=0.1 0.1 0.1
- added link Head_visual_ears; visual mesh filename=meshes/pepper_1.7/HeadPitch_ears.obj scale=0.1 0.1 0.1
- added link Head_visual_milky; visual mesh filename=meshes/pepper_1.7/HeadPitch_face_milky.obj scale=0.1 0.1 0.1
- added link Torso_visual_shiny; visual mesh filename=meshes/pepper_1.7/Torso_shiny.obj scale=0.1 0.1 0.1
- added link Torso_visual_transparent; visual mesh filename=meshes/pepper_1.7/Torso_transparent.obj scale=0.1 0.1 0.1
- link Head: geometry collision mesh filename=meshes/pepper_1.7/HeadPitch_0.10.stl scale=0.1 0.1 0.1; visual mesh filename=meshes/pepper_1.7/HeadPitch_eyes.obj scale=0.1 0.1 0.1
- link r_wrist: geometry collision mesh filename=meshes/pepper_1.7/RWristYaw_0.10.stl scale=0.1 0.1 0.1; visual mesh filename=meshes/pepper_1.7/RWristYaw.obj scale=0.1 0.1 0.1
- link torso: geometry collision mesh filename=meshes/pepper_1.7/Torso_0.10.stl scale=0.1 0.1 0.1; visual mesh filename=meshes/pepper_1.7/Torso_milky.obj scale=0.1 0.1 0.1
Joints:
- added joint HeadPitch_face_shiny_joint: type fixed, parent Head, child HeadPitch_face_shiny, origin xyz=0 0 0 rpy=0 0 0
- added joint Head_visual_ears_joint: type fixed, parent Head, child Head_visual_ears, origin xyz=0 0 0 rpy=0 0 0
- added joint Head_visual_milky_joint: type fixed, parent Head, child Head_visual_milky, origin xyz=0 0 0 rpy=0 0 0
- added joint Torso_visual_shiny_joint: type fixed, parent torso, child Torso_visual_shiny, origin xyz=0 0 0 rpy=0 0 0
- added joint Torso_visual_transparent_joint: type fixed, parent torso, child Torso_visual_transparent, origin xyz=0 0 0 rpy=0 0 0

Commit message: Add HeadYaw, neck of the robot

File: urdf/pepper_1.7/pepper.urdf (robot description, URDF)
Before this commit: robot JulietteY20MP, 87 links, 86 joints
Links:
- link Neck: geometry collision mesh filename=meshes/pepper_1.7/HeadYaw_0.10.stl scale=0.1 0.1 0.1; visual mesh filename=meshes/pepper_1.7/HeadYaw.obj scale=0.1 0.1 0.1
- link r_wrist: geometry collision mesh filename=meshes/pepper_1.7/RWristYaw_0.10.stl scale=0.1 0.1 0.1; visual mesh filename=meshes/pepper_1.7/RWristYaw.dae scale=0.1 0.1 0.1

Commit message: Add HipPitch with textures

File: urdf/pepper_1.7/pepper.urdf (robot description, URDF)
Before this commit: robot JulietteY20MP, 87 links, 86 joints
Links:
- added link HipPitch_shiny; visual mesh filename=meshes/pepper_1.7/HipPitch_shiny.obj scale=0.1 0.1 0.1
- link Pelvis: geometry collision mesh filename=meshes/pepper_1.7/HipPitch_0.10.stl scale=0.1 0.1 0.1; visual mesh filename=meshes/pepper_1.7/HipPitch_milky.obj scale=0.1 0.1 0.1
Joints:
- added joint HipPitch_shiny_joint: type fixed, parent Hip, child HipPitch_shiny, origin xyz=0 0 0 rpy=0 0 0

Commit message: Add HipRoll with texture

File: urdf/pepper_1.7/pepper.urdf (robot description, URDF)
Before this commit: robot JulietteY20MP, 88 links, 87 joints
Links:
- link Hip: geometry collision mesh filename=meshes/pepper_1.7/HipRoll_0.10.stl scale=0.1 0.1 0.1; visual mesh filename=meshes/pepper_1.7/HipRoll.obj scale=0.1 0.1 0.1

Commit message: Update KneePitch with texture

File: urdf/pepper_1.7/pepper.urdf (robot description, URDF)
Before this commit: robot JulietteY20MP, 88 links, 87 joints
Links:
- added link KneePitch_milky; visual mesh filename=meshes/pepper_1.7/KneePitch_milky.obj scale=0.1 0.1 0.1
- link Tibia: geometry collision mesh filename=meshes/pepper_1.7/KneePitch_0.10.stl scale=0.1 0.1 0.1; visual mesh filename=meshes/pepper_1.7/KneePitch_shiny.obj scale=0.1 0.1 0.1
Joints:
- added joint KneePitch_milky_joint: type fixed, parent Tibia, child KneePitch_milky, origin xyz=0 0 0 rpy=0 0 0

Commit message: Textured ElbowRoll

File: urdf/pepper_1.7/pepper.urdf (robot description, URDF)
Before this commit: robot JulietteY20MP, 89 links, 88 joints
Links:
- added link LElbowRoll_milky; visual mesh filename=meshes/pepper_1.7/LElbowRoll_milky.obj scale=0.1 0.1 0.1
- link LForeArm: geometry collision mesh filename=meshes/pepper_1.7/LElbowRoll_0.10.stl scale=0.1 0.1 0.1; visual mesh filename=meshes/pepper_1.7/LElbowRoll_shiny.obj scale=0.1 0.1 0.1
Joints:
- added joint LElbowRoll_milky_joint: type fixed, parent LElbow, child LElbowRoll_milky, origin xyz=0 0 0 rpy=0 0 0

Commit message: Textured LElbowYaw

File: urdf/pepper_1.7/pepper.urdf (robot description, URDF)
Before this commit: robot JulietteY20MP, 90 links, 89 joints
Links:
- link LElbow: geometry collision mesh filename=meshes/pepper_1.7/LElbowYaw_0.10.stl scale=0.1 0.1 0.1; visual mesh filename=meshes/pepper_1.7/LElbowYaw.obj scale=0.1 0.1 0.1

Commit message: LFingers and LShoulderPitch with textures

File: urdf/pepper_1.7/pepper.urdf (robot description, URDF)
Before this commit: robot JulietteY20MP, 90 links, 89 joints
Links:
- link LFinger11_link: geometry collision mesh filename=meshes/pepper_1.7/LFinger11_0.10.stl scale=0.1 0.1 0.1; visual mesh filename=meshes/pepper_1.7/LFinger11.obj scale=0.1 0.1 0.1
- link LFinger12_link: geometry collision mesh filename=meshes/pepper_1.7/LFinger12_0.10.stl scale=0.1 0.1 0.1; visual mesh filename=meshes/pepper_1.7/LFinger12.obj scale=0.1 0.1 0.1
- link LFinger13_link: geometry collision mesh filename=meshes/pepper_1.7/LFinger13_0.10.stl scale=0.1 0.1 0.1; visual mesh filename=meshes/pepper_1.7/LFinger13.obj scale=0.1 0.1 0.1
- link LFinger21_link: geometry collision mesh filename=meshes/pepper_1.7/LFinger21_0.10.stl scale=0.1 0.1 0.1; visual mesh filename=meshes/pepper_1.7/LFinger21.obj scale=0.1 0.1 0.1
- link LFinger22_link: geometry collision mesh filename=meshes/pepper_1.7/LFinger22_0.10.stl scale=0.1 0.1 0.1; visual mesh filename=meshes/pepper_1.7/LFinger22.obj scale=0.1 0.1 0.1
- link LFinger23_link: geometry collision mesh filename=meshes/pepper_1.7/LFinger23_0.10.stl scale=0.1 0.1 0.1; visual mesh filename=meshes/pepper_1.7/LFinger23.obj scale=0.1 0.1 0.1
- link LFinger31_link: geometry collision mesh filename=meshes/pepper_1.7/LFinger31_0.10.stl scale=0.1 0.1 0.1; visual mesh filename=meshes/pepper_1.7/LFinger31.obj scale=0.1 0.1 0.1
- link LFinger32_link: geometry collision mesh filename=meshes/pepper_1.7/LFinger32_0.10.stl scale=0.1 0.1 0.1; visual mesh filename=meshes/pepper_1.7/LFinger32.obj scale=0.1 0.1 0.1
- link LFinger33_link: geometry collision mesh filename=meshes/pepper_1.7/LFinger33_0.10.stl scale=0.1 0.1 0.1; visual mesh filename=meshes/pepper_1.7/LFinger33.obj scale=0.1 0.1 0.1
- link LFinger41_link: geometry collision mesh filename=meshes/pepper_1.7/LFinger41_0.10.stl scale=0.1 0.1 0.1; visual mesh filename=meshes/pepper_1.7/LFinger41.obj scale=0.1 0.1 0.1
- link LFinger42_link: geometry collision mesh filename=meshes/pepper_1.7/LFinger42_0.10.stl scale=0.1 0.1 0.1; visual mesh filename=meshes/pepper_1.7/LFinger42.obj scale=0.1 0.1 0.1
- link LFinger43_link: geometry collision mesh filename=meshes/pepper_1.7/LFinger43_0.10.stl scale=0.1 0.1 0.1; visual mesh filename=meshes/pepper_1.7/LFinger43.obj scale=0.1 0.1 0.1
- link LShoulder: geometry collision mesh filename=meshes/pepper_1.7/LShoulderPitch_0.10.stl scale=0.1 0.1 0.1; visual mesh filename=meshes/pepper_1.7/LShoulderPitch.obj scale=0.1 0.1 0.1

Commit message: Add LShoulderRoll textured

File: urdf/pepper_1.7/pepper.urdf (robot description, URDF)
Before this commit: robot JulietteY20MP, 90 links, 89 joints
Links:
- added link LShoulderRoll_shiny; visual mesh filename=meshes/pepper_1.7/LShoulderRoll_shiny.obj scale=0.1 0.1 0.1
- link LBicep: geometry collision mesh filename=meshes/pepper_1.7/LShoulderRoll_0.10.stl scale=0.1 0.1 0.1; visual mesh filename=meshes/pepper_1.7/LShoulderRoll_milky.obj scale=0.1 0.1 0.1
Joints:
- added joint LShoulderRoll_shiny_joint: type fixed, parent LShoulder, child LShoulderRoll_shiny, origin xyz=0 0 0 rpy=0 0 0

Commit message: Additional textured links

File: urdf/pepper_1.7/pepper.urdf (robot description, URDF)
Before this commit: robot JulietteY20MP, 91 links, 90 joints
Links:
- added link RElbowRoll_milky; visual mesh filename=meshes/pepper_1.7/RElbowRoll_milky.obj scale=0.1 0.1 0.1
- link LThumb1_link: geometry collision mesh filename=meshes/pepper_1.7/LThumb1_0.10.stl scale=0.1 0.1 0.1; visual mesh filename=meshes/pepper_1.7/LThumb1.obj scale=0.1 0.1 0.1
- link LThumb2_link: geometry collision mesh filename=meshes/pepper_1.7/LThumb2_0.10.stl scale=0.1 0.1 0.1; visual mesh filename=meshes/pepper_1.7/LThumb2.obj scale=0.1 0.1 0.1
- link RForeArm: geometry collision mesh filename=meshes/pepper_1.7/RElbowRoll_0.10.stl scale=0.1 0.1 0.1; visual mesh filename=meshes/pepper_1.7/RElbowRoll_shiny.obj scale=0.1 0.1 0.1
- link l_wrist: geometry collision mesh filename=meshes/pepper_1.7/LWristYaw_0.10.stl scale=0.1 0.1 0.1; visual mesh filename=meshes/pepper_1.7/LWristYaw.obj scale=0.1 0.1 0.1
Joints:
- added joint RElbowRoll_milky_joint: type fixed, parent RElbow, child RElbowRoll_milky, origin xyz=0 0 0 rpy=0 0 0

Commit message: Update links

File: urdf/pepper_1.7/pepper.urdf (robot description, URDF)
Before this commit: robot JulietteY20MP, 92 links, 91 joints
Links:
- link RElbow: geometry collision mesh filename=meshes/pepper_1.7/RElbowYaw_0.10.stl scale=0.1 0.1 0.1; visual mesh filename=meshes/pepper_1.7/RElbowYaw.obj scale=0.1 0.1 0.1
- link RFinger11_link: geometry collision mesh filename=meshes/pepper_1.7/RFinger11_0.10.stl scale=0.1 0.1 0.1; visual mesh filename=meshes/pepper_1.7/RFinger11.obj scale=0.1 0.1 0.1

Commit message: Add additional textured links

File: urdf/pepper_1.7/pepper.urdf (robot description, URDF)
Before this commit: robot JulietteY20MP, 92 links, 91 joints
Links:
- removed link HeadPitch_face_shiny
- removed link Head_visual_ears
- removed link Head_visual_milky
- removed link Torso_visual_shiny
- removed link Torso_visual_transparent
- added link HeadPitch_ears; visual mesh filename=meshes/pepper_1.7/HeadPitch_ears.obj scale=0.1 0.1 0.1
- added link HeadPitch_milky; visual mesh filename=meshes/pepper_1.7/HeadPitch_milky.obj scale=0.1 0.1 0.1
- added link HeadPitch_shiny; visual mesh filename=meshes/pepper_1.7/HeadPitch_shiny.obj scale=0.1 0.1 0.1
- added link RShoulderRoll_shiny; visual mesh filename=meshes/pepper_1.7/RShoulderRoll_shiny.obj scale=0.1 0.1 0.1
- added link Torso_shiny; visual mesh filename=meshes/pepper_1.7/Torso_shiny.obj scale=0.1 0.1 0.1
- added link Torso_transparent; visual mesh filename=meshes/pepper_1.7/Torso_transparent.obj scale=0.1 0.1 0.1
- link RBicep: geometry collision mesh filename=meshes/pepper_1.7/RShoulderRoll_0.10.stl scale=0.1 0.1 0.1; visual mesh filename=meshes/pepper_1.7/RShoulderRoll_milky.obj scale=0.1 0.1 0.1
- link RFinger12_link: geometry collision mesh filename=meshes/pepper_1.7/RFinger12_0.10.stl scale=0.1 0.1 0.1; visual mesh filename=meshes/pepper_1.7/RFinger12.obj scale=0.1 0.1 0.1
- link RFinger13_link: geometry collision mesh filename=meshes/pepper_1.7/RFinger13_0.10.stl scale=0.1 0.1 0.1; visual mesh filename=meshes/pepper_1.7/RFinger13.obj scale=0.1 0.1 0.1
- link RFinger21_link: geometry collision mesh filename=meshes/pepper_1.7/RFinger21_0.10.stl scale=0.1 0.1 0.1; visual mesh filename=meshes/pepper_1.7/RFinger21.obj scale=0.1 0.1 0.1
- link RFinger22_link: geometry collision mesh filename=meshes/pepper_1.7/RFinger22_0.10.stl scale=0.1 0.1 0.1; visual mesh filename=meshes/pepper_1.7/RFinger22.obj scale=0.1 0.1 0.1
- link RFinger23_link: geometry collision mesh filename=meshes/pepper_1.7/RFinger23_0.10.stl scale=0.1 0.1 0.1; visual mesh filename=meshes/pepper_1.7/RFinger23.obj scale=0.1 0.1 0.1
- link RFinger31_link: geometry collision mesh filename=meshes/pepper_1.7/RFinger31_0.10.stl scale=0.1 0.1 0.1; visual mesh filename=meshes/pepper_1.7/RFinger31.obj scale=0.1 0.1 0.1
- link RFinger32_link: geometry collision mesh filename=meshes/pepper_1.7/RFinger32_0.10.stl scale=0.1 0.1 0.1; visual mesh filename=meshes/pepper_1.7/RFinger32.obj scale=0.1 0.1 0.1
- link RFinger33_link: geometry collision mesh filename=meshes/pepper_1.7/RFinger33_0.10.stl scale=0.1 0.1 0.1; visual mesh filename=meshes/pepper_1.7/RFinger33.obj scale=0.1 0.1 0.1
- link RFinger41_link: geometry collision mesh filename=meshes/pepper_1.7/RFinger41_0.10.stl scale=0.1 0.1 0.1; visual mesh filename=meshes/pepper_1.7/RFinger41.obj scale=0.1 0.1 0.1
- link RFinger42_link: geometry collision mesh filename=meshes/pepper_1.7/RFinger42_0.10.stl scale=0.1 0.1 0.1; visual mesh filename=meshes/pepper_1.7/RFinger42.obj scale=0.1 0.1 0.1
- link RFinger43_link: geometry collision mesh filename=meshes/pepper_1.7/RFinger43_0.10.stl scale=0.1 0.1 0.1; visual mesh filename=meshes/pepper_1.7/RFinger43.obj scale=0.1 0.1 0.1
- link RShoulder: geometry collision mesh filename=meshes/pepper_1.7/RShoulderPitch_0.10.stl scale=0.1 0.1 0.1; visual mesh filename=meshes/pepper_1.7/RShoulderPitch.obj scale=0.1 0.1 0.1
- link RThumb1_link: geometry collision mesh filename=meshes/pepper_1.7/RThumb1_0.10.stl scale=0.1 0.1 0.1; visual mesh filename=meshes/pepper_1.7/RThumb1.obj scale=0.1 0.1 0.1
- link RThumb2_link: geometry collision mesh filename=meshes/pepper_1.7/RThumb2_0.10.stl scale=0.1 0.1 0.1; visual mesh filename=meshes/pepper_1.7/RThumb2.obj scale=0.1 0.1 0.1
- link WheelB_link: geometry collision mesh filename=meshes/pepper_1.7/WheelB_0.10.stl scale=0.1 0.1 0.1; visual mesh filename=meshes/pepper_1.7/WheelB.obj scale=0.1 0.1 0.1
- link WheelFL_link: geometry collision mesh filename=meshes/pepper_1.7/WheelFL_0.10.stl scale=0.1 0.1 0.1; visual mesh filename=meshes/pepper_1.7/WheelFL.obj scale=0.1 0.1 0.1
- link WheelFR_link: geometry collision mesh filename=meshes/pepper_1.7/WheelFR_0.10.stl scale=0.1 0.1 0.1; visual mesh filename=meshes/pepper_1.7/WheelFR.obj scale=0.1 0.1 0.1
- link r_wrist: geometry collision mesh filename=meshes/pepper_1.7/RWristYaw_0.10.stl scale=0.1 0.1 0.1; visual mesh filename=meshes/pepper_1.7/RWristYaw.obj scale=0.1 0.1 0.1
Joints:
- removed joint HeadPitch_face_shiny_joint
- removed joint Head_visual_ears_joint
- removed joint Head_visual_milky_joint
- removed joint Torso_visual_shiny_joint
- removed joint Torso_visual_transparent_joint
- added joint HeadPitch_ears_joint: type fixed, parent Head, child HeadPitch_ears, origin xyz=0 0 0 rpy=0 0 0
- added joint HeadPitch_milky_joint: type fixed, parent Head, child HeadPitch_milky, origin xyz=0 0 0 rpy=0 0 0
- added joint HeadPitch_shiny_joint: type fixed, parent Head, child HeadPitch_shiny, origin xyz=0 0 0 rpy=0 0 0
- added joint RShoulderRoll_shiny_joint: type fixed, parent RShoulder, child RShoulderRoll_shiny, origin xyz=0 0 0 rpy=0 0 0
- added joint Torso_shiny_joint: type fixed, parent torso, child Torso_shiny, origin xyz=0 0 0 rpy=0 0 0
- added joint Torso_transparent_joint: type fixed, parent torso, child Torso_transparent, origin xyz=0 0 0 rpy=0 0 0

Commit message: Update URDF to avoid mesh display bug

File: urdf/pepper_1.7/pepper.urdf (robot description, URDF)
Before this commit: robot JulietteY20MP, 93 links, 92 joints
Joints:
- joint HipPitch_shiny_joint: parent Hip -> Pelvis
- joint LElbowRoll_milky_joint: parent LElbow -> LForeArm
- joint LShoulderRoll_shiny_joint: parent LShoulder -> LBicep
- joint RElbowRoll_milky_joint: parent RElbow -> RForeArm
- joint RShoulderRoll_shiny_joint: parent RShoulder -> RBicep

Commit message: Wheels test

File: urdf/pepper_1.7/pepper.urdf (robot description, URDF)
Before this commit: robot JulietteY20MP, 93 links, 92 joints
Links:
- added link Free_WheelB_link
- added link Free_WheelFL_link
- added link Free_WheelFR_link
Joints:
- added joint Free_WheelB: type continuous, parent WheelB_link, child Free_WheelB_link, origin xyz=0 0 0 rpy=0 0 0, axis 0.0 1.0 0.0
- added joint Free_WheelFL: type continuous, parent WheelFL_link, child Free_WheelFL_link, origin xyz=0 0 0 rpy=0 0 0, axis 0.0 1.0 0.0
- added joint Free_WheelFR: type continuous, parent WheelFR_link, child Free_WheelFR_link, origin xyz=0 0 0 rpy=0 0 0, axis 0.0 1.0 0.0
- joint WheelB: axis 1.0 0 0 -> 1.0 0.0 0.0; limit lower=0 upper=0 effort=3.25 velocity=6.28319 -> (none)
- joint WheelFL: limit lower=0 upper=0 effort=3.25 velocity=6.28319 -> (none)
- joint WheelFR: limit lower=0 upper=0 effort=3.25 velocity=6.28319 -> (none)

Commit message: Update URDF and wheel tests

File: urdf/pepper_1.7/pepper.urdf (robot description, URDF)
Before this commit: robot JulietteY20MP, 96 links, 95 joints
Links:
- removed link Free_WheelB_link
- removed link Free_WheelFL_link
- removed link Free_WheelFR_link
- link WheelB_link: geometry collision mesh filename=meshes/pepper_1.7/WheelB.obj scale=0.1 0.1 0.1; visual mesh filename=meshes/pepper_1.7/WheelB.obj scale=0.1 0.1 0.1
- link WheelFL_link: geometry collision mesh filename=meshes/pepper_1.7/WheelFL.obj scale=0.1 0.1 0.1; visual mesh filename=meshes/pepper_1.7/WheelFL.obj scale=0.1 0.1 0.1
- link WheelFR_link: geometry collision mesh filename=meshes/pepper_1.7/WheelFR.obj scale=0.1 0.1 0.1; visual mesh filename=meshes/pepper_1.7/WheelFR.obj scale=0.1 0.1 0.1
Joints:
- removed joint Free_WheelB
- removed joint Free_WheelFL
- removed joint Free_WheelFR
