Commit message: fix path nao meshes Signed-off-by: Maxime Caniot <mcaniot@aldebaran.com>

File: qibullet/robot_data/nao_V40/nao.urdf (robot description, URDF)
Before this commit: robot NaoH25V50, 79 links, 78 joints
Links:
- link Head: geometry collision mesh filename=meshes/HeadPitch_0.10.stl scale=0.1 0.1 0.1; visual mesh filename=meshes/HeadPitch_0.10.stl scale=0.1 0.1 0.1
- link LAnklePitch: geometry collision mesh filename=meshes/LAnklePitch_0.10.stl scale=0.1 0.1 0.1; visual mesh filename=meshes/LAnklePitch_0.10.stl scale=0.1 0.1 0.1
- link LBicep: geometry collision mesh filename=meshes/LShoulderRoll_0.10.stl scale=0.1 0.1 0.1; visual mesh filename=meshes/LShoulderRoll_0.10.stl scale=0.1 0.1 0.1
- link LFinger11_link: geometry collision mesh filename=meshes/LFinger11_0.10.stl scale=0.1 0.1 0.1; visual mesh filename=meshes/LFinger11_0.10.stl scale=0.1 0.1 0.1
- link LFinger12_link: geometry collision mesh filename=meshes/LFinger12_0.10.stl scale=0.1 0.1 0.1; visual mesh filename=meshes/LFinger12_0.10.stl scale=0.1 0.1 0.1
- link LFinger13_link: geometry collision mesh filename=meshes/LFinger13_0.10.stl scale=0.1 0.1 0.1; visual mesh filename=meshes/LFinger13_0.10.stl scale=0.1 0.1 0.1
- link LFinger21_link: geometry collision mesh filename=meshes/LFinger21_0.10.stl scale=0.1 0.1 0.1; visual mesh filename=meshes/LFinger21_0.10.stl scale=0.1 0.1 0.1
- link LFinger22_link: geometry collision mesh filename=meshes/LFinger22_0.10.stl scale=0.1 0.1 0.1; visual mesh filename=meshes/LFinger22_0.10.stl scale=0.1 0.1 0.1
- link LFinger23_link: geometry collision mesh filename=meshes/LFinger23_0.10.stl scale=0.1 0.1 0.1; visual mesh filename=meshes/LFinger23_0.10.stl scale=0.1 0.1 0.1
- link LForeArm: geometry collision mesh filename=meshes/LElbowRoll_0.10.stl scale=0.1 0.1 0.1; visual mesh filename=meshes/LElbowRoll_0.10.stl scale=0.1 0.1 0.1
- link LHip: geometry collision mesh filename=meshes/LHipRoll_0.10.stl scale=0.1 0.1 0.1; visual mesh filename=meshes/LHipRoll_0.10.stl scale=0.1 0.1 0.1
- link LPelvis: geometry collision mesh filename=meshes/LHipYawPitch_0.10.stl scale=0.1 0.1 0.1; visual mesh filename=meshes/LHipYawPitch_0.10.stl scale=0.1 0.1 0.1
- link LShoulder: geometry collision mesh filename=meshes/LShoulderPitch_0.10.stl scale=0.1 0.1 0.1; visual mesh filename=meshes/LShoulderPitch_0.10.stl scale=0.1 0.1 0.1
- link LThigh: geometry collision mesh filename=meshes/LHipPitch_0.10.stl scale=0.1 0.1 0.1; visual mesh filename=meshes/LHipPitch_0.10.stl scale=0.1 0.1 0.1
- link LThumb1_link: geometry collision mesh filename=meshes/LThumb1_0.10.stl scale=0.1 0.1 0.1; visual mesh filename=meshes/LThumb1_0.10.stl scale=0.1 0.1 0.1
- link LThumb2_link: geometry collision mesh filename=meshes/LThumb2_0.10.stl scale=0.1 0.1 0.1; visual mesh filename=meshes/LThumb2_0.10.stl scale=0.1 0.1 0.1
- link LTibia: geometry collision mesh filename=meshes/LKneePitch_0.10.stl scale=0.1 0.1 0.1; visual mesh filename=meshes/LKneePitch_0.10.stl scale=0.1 0.1 0.1
- link Neck: geometry collision mesh filename=meshes/HeadYaw_0.10.stl scale=0.1 0.1 0.1; visual mesh filename=meshes/HeadYaw_0.10.stl scale=0.1 0.1 0.1
- link RAnklePitch: geometry collision mesh filename=meshes/RAnklePitch_0.10.stl scale=0.1 0.1 0.1; visual mesh filename=meshes/RAnklePitch_0.10.stl scale=0.1 0.1 0.1
- link RBicep: geometry collision mesh filename=meshes/RShoulderRoll_0.10.stl scale=0.1 0.1 0.1; visual mesh filename=meshes/RShoulderRoll_0.10.stl scale=0.1 0.1 0.1
- link RFinger11_link: geometry collision mesh filename=meshes/RFinger11_0.10.stl scale=0.1 0.1 0.1; visual mesh filename=meshes/RFinger11_0.10.stl scale=0.1 0.1 0.1
- link RFinger12_link: geometry collision mesh filename=meshes/RFinger12_0.10.stl scale=0.1 0.1 0.1; visual mesh filename=meshes/RFinger12_0.10.stl scale=0.1 0.1 0.1
- link RFinger13_link: geometry collision mesh filename=meshes/RFinger13_0.10.stl scale=0.1 0.1 0.1; visual mesh filename=meshes/RFinger13_0.10.stl scale=0.1 0.1 0.1
- link RFinger21_link: geometry collision mesh filename=meshes/RFinger21_0.10.stl scale=0.1 0.1 0.1; visual mesh filename=meshes/RFinger21_0.10.stl scale=0.1 0.1 0.1
- link RFinger22_link: geometry collision mesh filename=meshes/RFinger22_0.10.stl scale=0.1 0.1 0.1; visual mesh filename=meshes/RFinger22_0.10.stl scale=0.1 0.1 0.1
- link RFinger23_link: geometry collision mesh filename=meshes/RFinger23_0.10.stl scale=0.1 0.1 0.1; visual mesh filename=meshes/RFinger23_0.10.stl scale=0.1 0.1 0.1
- link RForeArm: geometry collision mesh filename=meshes/RElbowRoll_0.10.stl scale=0.1 0.1 0.1; visual mesh filename=meshes/RElbowRoll_0.10.stl scale=0.1 0.1 0.1
- link RHip: geometry collision mesh filename=meshes/RHipRoll_0.10.stl scale=0.1 0.1 0.1; visual mesh filename=meshes/RHipRoll_0.10.stl scale=0.1 0.1 0.1
- link RPelvis: geometry collision mesh filename=meshes/RHipYawPitch_0.10.stl scale=0.1 0.1 0.1; visual mesh filename=meshes/RHipYawPitch_0.10.stl scale=0.1 0.1 0.1
- link RShoulder: geometry collision mesh filename=meshes/RShoulderPitch_0.10.stl scale=0.1 0.1 0.1; visual mesh filename=meshes/RShoulderPitch_0.10.stl scale=0.1 0.1 0.1
- link RThigh: geometry collision mesh filename=meshes/RHipPitch_0.10.stl scale=0.1 0.1 0.1; visual mesh filename=meshes/RHipPitch_0.10.stl scale=0.1 0.1 0.1
- link RThumb1_link: geometry collision mesh filename=meshes/RThumb1_0.10.stl scale=0.1 0.1 0.1; visual mesh filename=meshes/RThumb1_0.10.stl scale=0.1 0.1 0.1
- link RThumb2_link: geometry collision mesh filename=meshes/RThumb2_0.10.stl scale=0.1 0.1 0.1; visual mesh filename=meshes/RThumb2_0.10.stl scale=0.1 0.1 0.1
- link RTibia: geometry collision mesh filename=meshes/RKneePitch_0.10.stl scale=0.1 0.1 0.1; visual mesh filename=meshes/RKneePitch_0.10.stl scale=0.1 0.1 0.1
- link l_ankle: geometry collision mesh filename=meshes/LAnkleRoll_0.10.stl scale=0.1 0.1 0.1; visual mesh filename=meshes/LAnkleRoll_0.10.stl scale=0.1 0.1 0.1
- link l_wrist: geometry collision mesh filename=meshes/LWristYaw_0.10.stl scale=0.1 0.1 0.1; visual mesh filename=meshes/LWristYaw_0.10.stl scale=0.1 0.1 0.1
- link r_ankle: geometry collision mesh filename=meshes/RAnkleRoll_0.10.stl scale=0.1 0.1 0.1; visual mesh filename=meshes/RAnkleRoll_0.10.stl scale=0.1 0.1 0.1
- link r_wrist: geometry collision mesh filename=meshes/RWristYaw_0.10.stl scale=0.1 0.1 0.1; visual mesh filename=meshes/RWristYaw_0.10.stl scale=0.1 0.1 0.1
- link torso: geometry collision mesh filename=meshes/Torso_0.10.stl scale=0.1 0.1 0.1; visual mesh filename=meshes/Torso_0.10.stl scale=0.1 0.1 0.1

Commit message: Correct mass and inertia for ghost links

File: qibullet/robot_data/nao_V40/nao.urdf (robot description, URDF)
Before this commit: robot NaoH25V50, 79 links, 78 joints
Links:
- link CameraBottom_frame: mass None -> 0
- link CameraBottom_optical_frame: mass None -> 0
- link CameraTop_frame: mass None -> 0
- link CameraTop_optical_frame: mass None -> 0
- link ChestButton_frame: mass None -> 0
- link HeadTouchFront_frame: mass None -> 0
- link HeadTouchMiddle_frame: mass None -> 0
- link HeadTouchRear_frame: mass None -> 0
- link ImuTorsoAccelerometer_frame: mass None -> 0
- link ImuTorsoGyrometer_frame: mass None -> 0
- link LFootBumperLeft_frame: mass None -> 0
- link LFootBumperRight_frame: mass None -> 0
- link LHandTouchBack_frame: mass None -> 0
- link LHandTouchLeft_frame: mass None -> 0
- link LHandTouchRight_frame: mass None -> 0
- link LInfraRed_frame: mass None -> 0
- link LSonar_frame: mass None -> 0
- link RFootBumperLeft_frame: mass None -> 0
- link RFootBumperRight_frame: mass None -> 0
- link RHandTouchBack_frame: mass None -> 0
- link RHandTouchLeft_frame: mass None -> 0
- link RHandTouchRight_frame: mass None -> 0
- link RInfraRed_frame: mass None -> 0
- link RSonar_frame: mass None -> 0
- link base_link: mass None -> 0.0000000001
- link gaze: mass None -> 0
- link l_sole: mass None -> 0
- link r_sole: mass None -> 0

Commit message: Update visual to dae instead of stl

File: qibullet/robot_data/nao_V40/nao.urdf (robot description, URDF)
Before this commit: robot NaoH25V50, 79 links, 78 joints
Links:
- link Head: geometry collision mesh filename=meshes/HeadPitch_0.10.stl scale=0.1 0.1 0.1; visual mesh filename=meshes/HeadPitch.dae scale=0.1 0.1 0.1
- link LAnklePitch: geometry collision mesh filename=meshes/LAnklePitch_0.10.stl scale=0.1 0.1 0.1; visual mesh filename=meshes/LAnklePitch.dae scale=0.1 0.1 0.1
- link LBicep: geometry collision mesh filename=meshes/LShoulderRoll_0.10.stl scale=0.1 0.1 0.1; visual mesh filename=meshes/LShoulderRoll.dae scale=0.1 0.1 0.1
- link LFinger11_link: geometry collision mesh filename=meshes/LFinger11_0.10.stl scale=0.1 0.1 0.1; visual mesh filename=meshes/LFinger11.dae scale=0.1 0.1 0.1
- link LFinger12_link: geometry collision mesh filename=meshes/LFinger12_0.10.stl scale=0.1 0.1 0.1; visual mesh filename=meshes/LFinger12.dae scale=0.1 0.1 0.1
- link LFinger13_link: geometry collision mesh filename=meshes/LFinger13_0.10.stl scale=0.1 0.1 0.1; visual mesh filename=meshes/LFinger13.dae scale=0.1 0.1 0.1
- link LFinger21_link: geometry collision mesh filename=meshes/LFinger21_0.10.stl scale=0.1 0.1 0.1; visual mesh filename=meshes/LFinger21.dae scale=0.1 0.1 0.1
- link LFinger22_link: geometry collision mesh filename=meshes/LFinger22_0.10.stl scale=0.1 0.1 0.1; visual mesh filename=meshes/LFinger22.dae scale=0.1 0.1 0.1
- link LFinger23_link: geometry collision mesh filename=meshes/LFinger23_0.10.stl scale=0.1 0.1 0.1; visual mesh filename=meshes/LFinger23.dae scale=0.1 0.1 0.1
- link LForeArm: geometry collision mesh filename=meshes/LElbowRoll_0.10.stl scale=0.1 0.1 0.1; visual mesh filename=meshes/LElbowRoll.dae scale=0.1 0.1 0.1
- link LHip: geometry collision mesh filename=meshes/LHipRoll_0.10.stl scale=0.1 0.1 0.1; visual mesh filename=meshes/LHipRoll.dae scale=0.1 0.1 0.1
- link LPelvis: geometry collision mesh filename=meshes/LHipYawPitch.dae scale=0.1 0.1 0.1; visual mesh filename=meshes/LHipYawPitch.dae scale=0.1 0.1 0.1
- link LShoulder: geometry collision mesh filename=meshes/LShoulderPitch_0.10.stl scale=0.1 0.1 0.1; visual mesh filename=meshes/LShoulderPitch.dae scale=0.1 0.1 0.1
- link LThigh: geometry collision mesh filename=meshes/LHipPitch_0.10.stl scale=0.1 0.1 0.1; visual mesh filename=meshes/LHipPitch.dae scale=0.1 0.1 0.1
- link LThumb1_link: geometry collision mesh filename=meshes/LThumb1_0.10.stl scale=0.1 0.1 0.1; visual mesh filename=meshes/LThumb1.dae scale=0.1 0.1 0.1
- link LThumb2_link: geometry collision mesh filename=meshes/LThumb2_0.10.stl scale=0.1 0.1 0.1; visual mesh filename=meshes/LThumb2.dae scale=0.1 0.1 0.1
- link LTibia: geometry collision mesh filename=meshes/LKneePitch_0.10.stl scale=0.1 0.1 0.1; visual mesh filename=meshes/LKneePitch.dae scale=0.1 0.1 0.1
- link Neck: geometry collision mesh filename=meshes/HeadYaw.dae scale=0.1 0.1 0.1; visual mesh filename=meshes/HeadYaw.dae scale=0.1 0.1 0.1
- link RAnklePitch: geometry collision mesh filename=meshes/RAnklePitch_0.10.stl scale=0.1 0.1 0.1; visual mesh filename=meshes/RAnklePitch.dae scale=0.1 0.1 0.1
- link RBicep: geometry collision mesh filename=meshes/RShoulderRoll_0.10.stl scale=0.1 0.1 0.1; visual mesh filename=meshes/RShoulderRoll.dae scale=0.1 0.1 0.1
- link RFinger11_link: geometry collision mesh filename=meshes/RFinger11_0.10.stl scale=0.1 0.1 0.1; visual mesh filename=meshes/RFinger11.dae scale=0.1 0.1 0.1
- link RFinger12_link: geometry collision mesh filename=meshes/RFinger12_0.10.stl scale=0.1 0.1 0.1; visual mesh filename=meshes/RFinger12.dae scale=0.1 0.1 0.1
- link RFinger13_link: geometry collision mesh filename=meshes/RFinger13_0.10.stl scale=0.1 0.1 0.1; visual mesh filename=meshes/RFinger13.dae scale=0.1 0.1 0.1
- link RFinger21_link: geometry collision mesh filename=meshes/RFinger21_0.10.stl scale=0.1 0.1 0.1; visual mesh filename=meshes/RFinger21.dae scale=0.1 0.1 0.1
- link RFinger22_link: geometry collision mesh filename=meshes/RFinger22_0.10.stl scale=0.1 0.1 0.1; visual mesh filename=meshes/RFinger22.dae scale=0.1 0.1 0.1
- link RFinger23_link: geometry collision mesh filename=meshes/RFinger23_0.10.stl scale=0.1 0.1 0.1; visual mesh filename=meshes/RFinger23.dae scale=0.1 0.1 0.1
- link RForeArm: geometry collision mesh filename=meshes/RElbowRoll_0.10.stl scale=0.1 0.1 0.1; visual mesh filename=meshes/RElbowRoll.dae scale=0.1 0.1 0.1
- link RHip: geometry collision mesh filename=meshes/RHipRoll_0.10.stl scale=0.1 0.1 0.1; visual mesh filename=meshes/RHipRoll.dae scale=0.1 0.1 0.1
- link RPelvis: geometry collision mesh filename=meshes/RHipYawPitch_0.10.stl scale=0.1 0.1 0.1; visual mesh filename=meshes/RHipYawPitch.dae scale=0.1 0.1 0.1
- link RShoulder: geometry collision mesh filename=meshes/RShoulderPitch_0.10.stl scale=0.1 0.1 0.1; visual mesh filename=meshes/RShoulderPitch.dae scale=0.1 0.1 0.1
- link RThigh: geometry collision mesh filename=meshes/RHipPitch_0.10.stl scale=0.1 0.1 0.1; visual mesh filename=meshes/RHipPitch.dae scale=0.1 0.1 0.1
- link RThumb1_link: geometry collision mesh filename=meshes/RThumb1_0.10.stl scale=0.1 0.1 0.1; visual mesh filename=meshes/RThumb1.dae scale=0.1 0.1 0.1
- link RThumb2_link: geometry collision mesh filename=meshes/RThumb2_0.10.stl scale=0.1 0.1 0.1; visual mesh filename=meshes/RThumb2.dae scale=0.1 0.1 0.1
- link RTibia: geometry collision mesh filename=meshes/RKneePitch_0.10.stl scale=0.1 0.1 0.1; visual mesh filename=meshes/RKneePitch.dae scale=0.1 0.1 0.1
- link l_ankle: geometry collision mesh filename=meshes/LAnkleRoll_0.10.stl scale=0.1 0.1 0.1; visual mesh filename=meshes/LAnkleRoll.dae scale=0.1 0.1 0.1
- link l_wrist: geometry collision mesh filename=meshes/LWristYaw_0.10.stl scale=0.1 0.1 0.1; visual mesh filename=meshes/LWristYaw.dae scale=0.1 0.1 0.1
- link r_ankle: geometry collision mesh filename=meshes/RAnkleRoll_0.10.stl scale=0.1 0.1 0.1; visual mesh filename=meshes/RAnkleRoll.dae scale=0.1 0.1 0.1
- link r_wrist: geometry collision mesh filename=meshes/RWristYaw_0.10.stl scale=0.1 0.1 0.1; visual mesh filename=meshes/RWristYaw.dae scale=0.1 0.1 0.1
- link torso: geometry collision mesh filename=meshes/Torso_0.10.stl scale=0.1 0.1 0.1; visual mesh filename=meshes/Torso.dae scale=0.1 0.1 0.1

Commit message: Transform the dae meshes to obj and mtl

File: qibullet/robot_data/nao_V40/nao.urdf (robot description, URDF)
Before this commit: robot NaoH25V50, 79 links, 78 joints
Links:
- link Head: geometry collision mesh filename=meshes/HeadPitch_0.10.stl scale=0.1 0.1 0.1; visual mesh filename=meshes/HeadPitch.obj scale=0.1 0.1 0.1
- link LAnklePitch: geometry collision mesh filename=meshes/LAnklePitch_0.10.stl scale=0.1 0.1 0.1; visual mesh filename=meshes/LAnklePitch.obj scale=0.1 0.1 0.1
- link LBicep: geometry collision mesh filename=meshes/LShoulderRoll_0.10.stl scale=0.1 0.1 0.1; visual mesh filename=meshes/LShoulderRoll.obj scale=0.1 0.1 0.1
- link LFinger11_link: geometry collision mesh filename=meshes/LFinger11_0.10.stl scale=0.1 0.1 0.1; visual mesh filename=meshes/LFinger11.obj scale=0.1 0.1 0.1
- link LFinger12_link: geometry collision mesh filename=meshes/LFinger12_0.10.stl scale=0.1 0.1 0.1; visual mesh filename=meshes/LFinger12.obj scale=0.1 0.1 0.1
- link LFinger13_link: geometry collision mesh filename=meshes/LFinger13_0.10.stl scale=0.1 0.1 0.1; visual mesh filename=meshes/LFinger13.obj scale=0.1 0.1 0.1
- link LFinger21_link: geometry collision mesh filename=meshes/LFinger21_0.10.stl scale=0.1 0.1 0.1; visual mesh filename=meshes/LFinger21.obj scale=0.1 0.1 0.1
- link LFinger22_link: geometry collision mesh filename=meshes/LFinger22_0.10.stl scale=0.1 0.1 0.1; visual mesh filename=meshes/LFinger22.obj scale=0.1 0.1 0.1
- link LFinger23_link: geometry collision mesh filename=meshes/LFinger23_0.10.stl scale=0.1 0.1 0.1; visual mesh filename=meshes/LFinger23.obj scale=0.1 0.1 0.1
- link LForeArm: geometry collision mesh filename=meshes/LElbowRoll_0.10.stl scale=0.1 0.1 0.1; visual mesh filename=meshes/LElbowRoll.obj scale=0.1 0.1 0.1
- link LHip: geometry collision mesh filename=meshes/LHipRoll_0.10.stl scale=0.1 0.1 0.1; visual mesh filename=meshes/LHipRoll.obj scale=0.1 0.1 0.1
- link LPelvis: geometry collision mesh filename=meshes/LHipYawPitch.obj scale=0.1 0.1 0.1; visual mesh filename=meshes/LHipYawPitch.obj scale=0.1 0.1 0.1
- link LShoulder: geometry collision mesh filename=meshes/LShoulderPitch_0.10.stl scale=0.1 0.1 0.1; visual mesh filename=meshes/LShoulderPitch.obj scale=0.1 0.1 0.1
- link LThigh: geometry collision mesh filename=meshes/LHipPitch_0.10.stl scale=0.1 0.1 0.1; visual mesh filename=meshes/LHipPitch.obj scale=0.1 0.1 0.1
- link LThumb1_link: geometry collision mesh filename=meshes/LThumb1_0.10.stl scale=0.1 0.1 0.1; visual mesh filename=meshes/LThumb1.obj scale=0.1 0.1 0.1
- link LThumb2_link: geometry collision mesh filename=meshes/LThumb2_0.10.stl scale=0.1 0.1 0.1; visual mesh filename=meshes/LThumb2.obj scale=0.1 0.1 0.1
- link LTibia: geometry collision mesh filename=meshes/LKneePitch_0.10.stl scale=0.1 0.1 0.1; visual mesh filename=meshes/LKneePitch.obj scale=0.1 0.1 0.1
- link Neck: geometry collision mesh filename=meshes/HeadYaw.obj scale=0.1 0.1 0.1; visual mesh filename=meshes/HeadYaw.obj scale=0.1 0.1 0.1
- link RAnklePitch: geometry collision mesh filename=meshes/RAnklePitch_0.10.stl scale=0.1 0.1 0.1; visual mesh filename=meshes/RAnklePitch.obj scale=0.1 0.1 0.1
- link RBicep: geometry collision mesh filename=meshes/RShoulderRoll_0.10.stl scale=0.1 0.1 0.1; visual mesh filename=meshes/RShoulderRoll.obj scale=0.1 0.1 0.1
- link RFinger11_link: geometry collision mesh filename=meshes/RFinger11_0.10.stl scale=0.1 0.1 0.1; visual mesh filename=meshes/RFinger11.obj scale=0.1 0.1 0.1
- link RFinger12_link: geometry collision mesh filename=meshes/RFinger12_0.10.stl scale=0.1 0.1 0.1; visual mesh filename=meshes/RFinger12.obj scale=0.1 0.1 0.1
- link RFinger13_link: geometry collision mesh filename=meshes/RFinger13_0.10.stl scale=0.1 0.1 0.1; visual mesh filename=meshes/RFinger13.obj scale=0.1 0.1 0.1
- link RFinger21_link: geometry collision mesh filename=meshes/RFinger21_0.10.stl scale=0.1 0.1 0.1; visual mesh filename=meshes/RFinger21.obj scale=0.1 0.1 0.1
- link RFinger22_link: geometry collision mesh filename=meshes/RFinger22_0.10.stl scale=0.1 0.1 0.1; visual mesh filename=meshes/RFinger22.obj scale=0.1 0.1 0.1
- link RFinger23_link: geometry collision mesh filename=meshes/RFinger23_0.10.stl scale=0.1 0.1 0.1; visual mesh filename=meshes/RFinger23.obj scale=0.1 0.1 0.1
- link RForeArm: geometry collision mesh filename=meshes/RElbowRoll_0.10.stl scale=0.1 0.1 0.1; visual mesh filename=meshes/RElbowRoll.obj scale=0.1 0.1 0.1
- link RHip: geometry collision mesh filename=meshes/RHipRoll_0.10.stl scale=0.1 0.1 0.1; visual mesh filename=meshes/RHipRoll.obj scale=0.1 0.1 0.1
- link RPelvis: geometry collision mesh filename=meshes/RHipYawPitch_0.10.stl scale=0.1 0.1 0.1; visual mesh filename=meshes/RHipYawPitch.obj scale=0.1 0.1 0.1
- link RShoulder: geometry collision mesh filename=meshes/RShoulderPitch_0.10.stl scale=0.1 0.1 0.1; visual mesh filename=meshes/RShoulderPitch.obj scale=0.1 0.1 0.1
- link RThigh: geometry collision mesh filename=meshes/RHipPitch_0.10.stl scale=0.1 0.1 0.1; visual mesh filename=meshes/RHipPitch.obj scale=0.1 0.1 0.1
- link RThumb1_link: geometry collision mesh filename=meshes/RThumb1_0.10.stl scale=0.1 0.1 0.1; visual mesh filename=meshes/RThumb1.obj scale=0.1 0.1 0.1
- link RThumb2_link: geometry collision mesh filename=meshes/RThumb2_0.10.stl scale=0.1 0.1 0.1; visual mesh filename=meshes/RThumb2.obj scale=0.1 0.1 0.1
- link RTibia: geometry collision mesh filename=meshes/RKneePitch_0.10.stl scale=0.1 0.1 0.1; visual mesh filename=meshes/RKneePitch.obj scale=0.1 0.1 0.1
- link l_ankle: geometry collision mesh filename=meshes/LAnkleRoll_0.10.stl scale=0.1 0.1 0.1; visual mesh filename=meshes/LAnkleRoll.obj scale=0.1 0.1 0.1
- link l_wrist: geometry collision mesh filename=meshes/LWristYaw_0.10.stl scale=0.1 0.1 0.1; visual mesh filename=meshes/LWristYaw.obj scale=0.1 0.1 0.1
- link r_ankle: geometry collision mesh filename=meshes/RAnkleRoll_0.10.stl scale=0.1 0.1 0.1; visual mesh filename=meshes/RAnkleRoll.obj scale=0.1 0.1 0.1
- link r_wrist: geometry collision mesh filename=meshes/RWristYaw_0.10.stl scale=0.1 0.1 0.1; visual mesh filename=meshes/RWristYaw.obj scale=0.1 0.1 0.1
- link torso: geometry collision mesh filename=meshes/Torso_0.10.stl scale=0.1 0.1 0.1; visual mesh filename=meshes/Torso.obj scale=0.1 0.1 0.1

Commit message: Correct R fingers and thumb

File: qibullet/robot_data/nao_V40/nao.urdf (robot description, URDF)
Before this commit: robot NaoH25V50, 79 links, 78 joints
Joints:
- joint RThumb2: origin xyz=0.01436 0 0 rpy=0 0 -0.999899 -> xyz=0.01336 -0.0035 0 rpy=0 0 -0.999899

Commit message: Correct orientations and positions for the left fingers and thumbs

File: qibullet/robot_data/nao_V40/nao.urdf (robot description, URDF)
Before this commit: robot NaoH25V50, 79 links, 78 joints
Joints:
- joint LThumb2: origin xyz=0.01436 0 0 rpy=0 0 -0.999899 -> xyz=0.01236 -0.0015 0 rpy=0 0 -0.999899
- joint RThumb2: origin xyz=0.01336 -0.0035 0 rpy=0 0 -0.999899 -> xyz=0.01236 -0.0015 0 rpy=0 0 -0.999899
