Commit message: Change NAO hand joints from continuous to revolute
EFFORT applied by the phalanx to be updated

File: qibullet/robot_data/nao_V40/nao.urdf (robot description, URDF)
Before this commit: robot NaoH25V50, 79 links, 78 joints
Joints:
- joint LFinger11: limit (none) -> lower=0.0 upper=0.999899 effort=0.144 velocity=12.56; type continuous -> revolute
- joint LFinger12: limit (none) -> lower=0.0 upper=0.999899 effort=0.144 velocity=12.56; type continuous -> revolute
- joint LFinger13: limit (none) -> lower=0.0 upper=0.999899 effort=0.144 velocity=12.56; type continuous -> revolute
- joint LFinger21: limit (none) -> lower=0.0 upper=0.999899 effort=0.144 velocity=12.56; type continuous -> revolute
- joint LFinger22: limit (none) -> lower=0.0 upper=0.999899 effort=0.144 velocity=12.56; type continuous -> revolute
- joint LFinger23: limit (none) -> lower=0.0 upper=0.999899 effort=0.144 velocity=12.56; type continuous -> revolute
- joint LThumb1: limit (none) -> lower=0.0 upper=0.999899 effort=0.144 velocity=12.56; type continuous -> revolute
- joint LThumb2: limit (none) -> lower=0.0 upper=0.999899 effort=0.144 velocity=12.56; type continuous -> revolute
- joint RFinger11: limit (none) -> lower=0.0 upper=0.999899 effort=0.144 velocity=12.56; type continuous -> revolute
- joint RFinger12: limit (none) -> lower=0.0 upper=0.999899 effort=0.144 velocity=12.56; type continuous -> revolute
- joint RFinger13: limit (none) -> lower=0.0 upper=0.999899 effort=0.144 velocity=12.56; type continuous -> revolute
- joint RFinger21: limit (none) -> lower=0.0 upper=0.999899 effort=0.144 velocity=12.56; type continuous -> revolute
- joint RFinger22: limit (none) -> lower=0.0 upper=0.999899 effort=0.144 velocity=12.56; type continuous -> revolute
- joint RFinger23: limit (none) -> lower=0.0 upper=0.999899 effort=0.144 velocity=12.56; type continuous -> revolute
- joint RThumb1: limit (none) -> lower=0.0 upper=0.999899 effort=0.144 velocity=12.56; type continuous -> revolute
- joint RThumb2: limit (none) -> lower=0.0 upper=0.999899 effort=0.144 velocity=12.56; type continuous -> revolute
