Commit message: Comment FSR in Romeo URDF

File: qibullet/robot_data/romeo_H37/romeo.urdf (robot description, URDF)
Before this commit: robot RomeoH37, 97 links, 96 joints
Links:
- removed link LFsrFToeFrontLeft_frame
- removed link LFsrFToeFrontRight_frame
- removed link LFsrFToeRearLeft_frame
- removed link LFsrFToeRearRight_frame
- removed link LFsrFrontCenter_frame
- removed link LFsrHeelLeft_frame
- removed link LFsrHeelRight_frame
- removed link LFsrRearCenter_frame
- removed link RFsrFToeFrontLeft_frame
- removed link RFsrFToeFrontRight_frame
- removed link RFsrFToeRearLeft_frame
- removed link RFsrFToeRearRight_frame
- removed link RFsrFrontCenter_frame
- removed link RFsrHeelLeft_frame
- removed link RFsrHeelRight_frame
- removed link RFsrRearCenter_frame
Joints:
- removed joint LFoot/FSR/CenterFront_sensor_fixedjoint
- removed joint LFoot/FSR/CenterRear_sensor_fixedjoint
- removed joint LFoot/FSR/HeelLeft_sensor_fixedjoint
- removed joint LFoot/FSR/HeelRight_sensor_fixedjoint
- removed joint LFoot/FSR/ToeFrontLeft_sensor_fixedjoint
- removed joint LFoot/FSR/ToeFrontRight_sensor_fixedjoint
- removed joint LFoot/FSR/ToeRearLeft_sensor_fixedjoint
- removed joint LFoot/FSR/ToeRearRight_sensor_fixedjoint
- removed joint RFoot/FSR/CenterFront_sensor_fixedjoint
- removed joint RFoot/FSR/CenterRear_sensor_fixedjoint
- removed joint RFoot/FSR/HeelLeft_sensor_fixedjoint
- removed joint RFoot/FSR/HeelRight_sensor_fixedjoint
- removed joint RFoot/FSR/ToeFrontLeft_sensor_fixedjoint
- removed joint RFoot/FSR/ToeFrontRight_sensor_fixedjoint
- removed joint RFoot/FSR/ToeRearLeft_sensor_fixedjoint
- removed joint RFoot/FSR/ToeRearRight_sensor_fixedjoint

Commit message: Update efforts in URDF

File: qibullet/robot_data/romeo_H37/romeo.urdf (robot description, URDF)
Before this commit: robot RomeoH37, 81 links, 80 joints
Links:
- removed link Cap
Joints:
- removed joint Cap_joint
- joint HeadPitch: limit lower=-0.2571 upper=0.2971 effort=2.57 velocity=1.9 -> lower=-0.2571 upper=0.2971 effort=9.40 velocity=1.9
- joint HeadRoll: limit lower=-0.4887 upper=0.4887 effort=3.748 velocity=1.5 -> lower=-0.4887 upper=0.4887 effort=14.46 velocity=1.5
- joint LAnklePitch: limit lower=-0.5149 upper=0.7505 effort=25.76 velocity=2.1 -> lower=-0.5149 upper=0.7505 effort=213.15 velocity=2.1
- joint LAnkleRoll: limit lower=-0.3491 upper=0.3491 effort=25.76 velocity=2.1 -> lower=-0.3491 upper=0.3491 effort=213.15 velocity=2.1
- joint LElbowRoll: limit lower=-2.2148 upper=1.9042 effort=7.404 velocity=3.7 -> lower=-2.2148 upper=1.9042 effort=13.86 velocity=3.7
- joint LElbowYaw: limit lower=-1.5228 upper=0.0044 effort=6.02 velocity=4.0 -> lower=-1.5228 upper=0.0044 effort=15.16 velocity=4.0
- joint LEyePitch: limit lower=-0.349066 upper=0.349066 effort=0.01752 velocity=293.215 -> lower=-0.349066 upper=0.349066 effort=1.752 velocity=293.215
- joint LEyeYaw: limit lower=-0.523599 upper=0.523599 effort=0.01752 velocity=293.215 -> lower=-0.523599 upper=0.523599 effort=1.752 velocity=293.215
- joint LFinger11: limit (none) -> lower=0.0 upper=0.988205 effort=0.91 velocity=59.8925
- joint LFinger12: limit (none) -> lower=0.0 upper=0.988205 effort=0.91 velocity=59.8925
- joint LFinger13: limit (none) -> lower=0.0 upper=0.988205 effort=0.91 velocity=59.8925
- joint LFinger21: limit (none) -> lower=0.0 upper=0.988205 effort=0.91 velocity=59.8925
- joint LFinger22: limit (none) -> lower=0.0 upper=0.988205 effort=0.91 velocity=59.8925
- joint LFinger23: limit (none) -> lower=0.0 upper=0.988205 effort=0.91 velocity=59.8925
- joint LFinger31: limit (none) -> lower=0.0 upper=0.988205 effort=0.91 velocity=59.8925
- joint LFinger32: limit (none) -> lower=0.0 upper=0.988205 effort=0.91 velocity=59.8925
- joint LFinger33: limit (none) -> lower=0.0 upper=0.988205 effort=0.91 velocity=59.8925
- joint LHipPitch: limit lower=-1.6581 upper=0.4014 effort=46.6 velocity=2.09 -> lower=-1.6581 upper=0.4014 effort=213.15 velocity=2.09
- joint LHipRoll: limit lower=-0.2618 upper=0.5236 effort=46.6 velocity=2.09 -> lower=-0.2618 upper=0.5236 effort=213.15 velocity=2.09
- joint LHipYaw: limit lower=-0.2618 upper=0.2618 effort=25.42 velocity=1.045 -> lower=-0.2618 upper=0.2618 effort=103.03 velocity=1.045
- joint LKneePitch: limit lower=-0.0218 upper=1.9722 effort=38.17 velocity=6.0 -> lower=-0.0218 upper=1.9722 effort=292.50 velocity=6.0
- joint LShoulderPitch: limit lower=-1.3491 upper=2.2462 effort=19.095 velocity=2.2 -> lower=-1.3491 upper=2.2462 effort=21.94 velocity=2.2
- joint LShoulderYaw: limit lower=-0.5768 upper=0.9242 effort=9.031 velocity=4.0 -> lower=-0.5768 upper=0.9242 effort=15.16 velocity=4.0
- joint LThumb1: limit (none) -> lower=0.0 upper=1.74533 effort=0.91 velocity=59.8925
- joint LThumb2: limit (none) -> lower=0.0 upper=0.988205 effort=0.91 velocity=59.8925
- joint LThumb3: limit (none) -> lower=0.0 upper=0.988205 effort=0.91 velocity=59.8925
- joint LWristPitch: limit lower=-0.988 upper=0.8969 effort=0.6 velocity=3.75 -> lower=-0.988 upper=0.8969 effort=1.39 velocity=3.75
- joint LWristRoll: limit lower=-3.6303 upper=0.4887 effort=2.177 velocity=1.1 -> lower=-3.6303 upper=0.4887 effort=7.23 velocity=1.1
- joint LWristYaw: limit lower=-0.4014 upper=0.4014 effort=0.862 velocity=2.26 -> lower=-0.4014 upper=0.4014 effort=2.01 velocity=2.26
- joint NeckPitch: limit lower=-0.3142 upper=0.6632 effort=5.956 velocity=2.2 -> lower=-0.3142 upper=0.6632 effort=35.0 velocity=2.2
- joint NeckYaw: limit lower=-2.0595 upper=2.0595 effort=7.324 velocity=4.0 -> lower=-2.0595 upper=2.0595 effort=27.72 velocity=4.0
- joint RAnklePitch: limit lower=-0.5149 upper=0.7505 effort=25.76 velocity=2.1 -> lower=-0.5149 upper=0.7505 effort=213.15 velocity=2.1
- joint RAnkleRoll: limit lower=-0.3491 upper=0.3491 effort=25.76 velocity=2.1 -> lower=-0.3491 upper=0.3491 effort=213.15 velocity=2.1
- joint RElbowRoll: limit lower=-1.9047 upper=2.2143 effort=7.404 velocity=3.7 -> lower=-1.9047 upper=2.2143 effort=13.86 velocity=3.7
- joint RElbowYaw: limit lower=-0.0047 upper=1.5225 effort=6.02 velocity=4.0 -> lower=-0.0047 upper=1.5225 effort=15.16 velocity=4.0
- joint REyePitch: limit lower=-0.349066 upper=0.349066 effort=0.01752 velocity=293.215 -> lower=-0.349066 upper=0.349066 effort=1.752 velocity=293.215
- joint REyeYaw: limit lower=-0.523599 upper=0.523599 effort=0.01752 velocity=293.215 -> lower=-0.523599 upper=0.523599 effort=1.752 velocity=293.215
- joint RFinger11: limit (none) -> lower=0.0 upper=0.988205 effort=0.91 velocity=59.8925
- joint RFinger12: limit (none) -> lower=0.0 upper=0.988205 effort=0.91 velocity=59.8925
- joint RFinger13: limit (none) -> lower=0.0 upper=0.988205 effort=0.91 velocity=59.8925
- joint RFinger21: limit (none) -> lower=0.0 upper=0.988205 effort=0.91 velocity=59.8925
- joint RFinger22: limit (none) -> lower=0.0 upper=0.988205 effort=0.91 velocity=59.8925
- joint RFinger23: limit (none) -> lower=0.0 upper=0.988205 effort=0.91 velocity=59.8925
- joint RFinger31: limit (none) -> lower=0.0 upper=0.988205 effort=0.91 velocity=59.8925
- joint RFinger32: limit (none) -> lower=0.0 upper=0.988205 effort=0.91 velocity=59.8925
- joint RFinger33: limit (none) -> lower=0.0 upper=0.988205 effort=0.91 velocity=59.8925
- joint RHipPitch: limit lower=-1.6581 upper=0.4014 effort=46.6 velocity=2.09 -> lower=-1.6581 upper=0.4014 effort=213.15 velocity=2.09
- joint RHipRoll: limit lower=-0.5236 upper=0.2618 effort=46.6 velocity=2.09 -> lower=-0.5236 upper=0.2618 effort=213.15 velocity=2.09
- joint RHipYaw: limit lower=-0.2618 upper=0.2618 effort=25.42 velocity=1.045 -> lower=-0.2618 upper=0.2618 effort=103.03 velocity=1.045
- joint RKneePitch: limit lower=-0.0218 upper=1.9722 effort=38.17 velocity=6.0 -> lower=-0.0218 upper=1.9722 effort=292.50 velocity=6.0
- joint RShoulderPitch: limit lower=-1.4554 upper=2.1399 effort=19.095 velocity=2.2 -> lower=-1.4554 upper=2.1399 effort=21.94 velocity=2.2
- joint RShoulderYaw: limit lower=-1.0985 upper=0.4025 effort=9.031 velocity=4.0 -> lower=-1.0985 upper=0.4025 effort=15.16 velocity=4.0
- joint RThumb1: limit (none) -> lower=0.0 upper=1.74533 effort=0.91 velocity=59.8925
- joint RThumb2: limit (none) -> lower=0.0 upper=0.988205 effort=0.91 velocity=59.8925
- joint RThumb3: limit (none) -> lower=0.0 upper=0.988205 effort=0.91 velocity=59.8925
- joint RWristPitch: limit lower=-0.9868 upper=0.8981 effort=0.6 velocity=3.75 -> lower=-0.9868 upper=0.8981 effort=1.39 velocity=3.75
- joint RWristRoll: limit lower=-0.4887 upper=3.6303 effort=2.177 velocity=1.1 -> lower=-0.4887 upper=3.6303 effort=7.23 velocity=1.1
- joint RWristYaw: limit lower=-0.4014 upper=0.4014 effort=0.862 velocity=2.26 -> lower=-0.4014 upper=0.4014 effort=2.01 velocity=2.26
- joint TrunkYaw: limit lower=-0.7575 upper=0.7575 effort=28.021 velocity=1.5 -> lower=-0.7575 upper=0.7575 effort=49.93 velocity=1.5

Commit message: Pass finger and thumb joints from continuous to revolute

File: qibullet/robot_data/romeo_H37/romeo.urdf (robot description, URDF)
Before this commit: robot RomeoH37, 80 links, 79 joints
Joints:
- joint LFinger11: type continuous -> revolute
- joint LFinger12: type continuous -> revolute
- joint LFinger13: type continuous -> revolute
- joint LFinger21: type continuous -> revolute
- joint LFinger22: type continuous -> revolute
- joint LFinger23: type continuous -> revolute
- joint LFinger31: type continuous -> revolute
- joint LFinger32: type continuous -> revolute
- joint LFinger33: type continuous -> revolute
- joint LThumb1: type continuous -> revolute
- joint LThumb2: type continuous -> revolute
- joint LThumb3: type continuous -> revolute
- joint RFinger11: type continuous -> revolute
- joint RFinger12: type continuous -> revolute
- joint RFinger13: type continuous -> revolute
- joint RFinger21: type continuous -> revolute
- joint RFinger22: type continuous -> revolute
- joint RFinger23: type continuous -> revolute
- joint RFinger31: type continuous -> revolute
- joint RFinger32: type continuous -> revolute
- joint RFinger33: type continuous -> revolute
- joint RThumb1: type continuous -> revolute
- joint RThumb2: type continuous -> revolute
- joint RThumb3: type continuous -> revolute

Commit message: Update mesh and urdf definition

File: qibullet/robot_data/romeo_H37/romeo.urdf (robot description, URDF)
Before this commit: robot RomeoH37, 80 links, 79 joints
Links:
- added link HeadRoll_logo, mass 0; visual mesh filename=meshes/HeadRoll_logo.obj scale=0.1 0.1 0.1
- added link HeadRoll_shell, mass 0; visual mesh filename=meshes/HeadRoll_shell.obj scale=0.1 0.1 0.1
- link HeadRoll_link: geometry collision mesh filename=meshes/HeadRoll_0.10.stl scale=1 1 1; visual mesh filename=meshes/HeadRoll_mainskin.obj scale=1 1 1
Joints:
- added joint HeadRoll_logo_joint: type fixed, parent HeadRoll_link, child HeadRoll_logo, origin xyz=0 0 0 rpy=0 0 0
- added joint HeadRoll_shell_joint: type fixed, parent HeadRoll_link, child HeadRoll_shell, origin xyz=0 0 0 rpy=0 0 0

Commit message: Mesh update

File: qibullet/robot_data/romeo_H37/romeo.urdf (robot description, URDF)
Before this commit: robot RomeoH37, 82 links, 81 joints
Links:
- added link LAnkleRoll_secondaryskin, mass 0; visual mesh filename=meshes/LAnkleRoll_secondaryskin.obj scale=1 1 1
- added link LAnkleRoll_secondaryskin2, mass 0; visual mesh filename=meshes/LAnkleRoll_secondaryskin2.obj scale=1 1 1
- added link LElbowYaw_shell, mass 0; visual mesh filename=meshes/LElbowYaw_shell.obj scale=1 1 1
- added link LHipPitch_flexibleskin, mass 0; visual mesh filename=meshes/LHipPitch_flexibleskin.obj scale=1 1 1
- added link LHipPitch_secondaryskin, mass 0; visual mesh filename=meshes/LHipPitch_secondaryskin.obj scale=1 1 1
- added link LHipPitch_shell, mass 0; visual mesh filename=meshes/LHipPitch_shell.obj scale=1 1 1
- added link LKneePitch_secondaryskin, mass 0; visual mesh filename=meshes/LKneePitch_secondaryskin.obj scale=1 1 1
- added link LKneePitch_secondaryskin2, mass 0; visual mesh filename=meshes/LKneePitch_secondaryskin2.obj scale=1 1 1
- added link LKneePitch_secondaryskin3, mass 0; visual mesh filename=meshes/LKneePitch_secondaryskin3.obj scale=1 1 1
- added link LKneePitch_shell, mass 0; visual mesh filename=meshes/LKneePitch_shell.obj scale=1 1 1
- added link LShoulderYaw_shell, mass 0; visual mesh filename=meshes/LShoulderYaw_shell.obj scale=1 1 1
- link HeadRoll_logo: geometry visual mesh filename=meshes/HeadRoll_logo.obj scale=1 1 1
- link HeadRoll_shell: geometry visual mesh filename=meshes/HeadRoll_shell.obj scale=1 1 1
- link LElbow: geometry collision mesh filename=meshes/LElbowYaw_0.10.stl scale=1 1 1; visual mesh filename=meshes/LElbowYaw_mainskin.obj scale=1 1 1
- link LEye: geometry collision mesh filename=meshes/LEyePitch_0.10.stl scale=1 1 1; visual mesh filename=meshes/LEyePitch.obj scale=1 1 1
- link LFinger11_link: geometry collision mesh filename=meshes/LFinger11_0.10.stl scale=1 1 1; visual mesh filename=meshes/LFinger11.obj scale=1 1 1
- link LFinger12_link: geometry collision mesh filename=meshes/LFinger12_0.10.stl scale=1 1 1; visual mesh filename=meshes/LFinger12.obj scale=1 1 1
- link LFinger13_link: geometry collision mesh filename=meshes/LFinger13_0.10.stl scale=1 1 1; visual mesh filename=meshes/LFinger13.obj scale=1 1 1
- link LFinger21_link: geometry collision mesh filename=meshes/LFinger21_0.10.stl scale=1 1 1; visual mesh filename=meshes/LFinger21.obj scale=1 1 1
- link LFinger22_link: geometry collision mesh filename=meshes/LFinger22_0.10.stl scale=1 1 1; visual mesh filename=meshes/LFinger22.obj scale=1 1 1
- link LFinger23_link: geometry collision mesh filename=meshes/LFinger23_0.10.stl scale=1 1 1; visual mesh filename=meshes/LFinger23.obj scale=1 1 1
- link LFinger31_link: geometry collision mesh filename=meshes/LFinger31_0.10.stl scale=1 1 1; visual mesh filename=meshes/LFinger31.obj scale=1 1 1
- link LFinger32_link: geometry collision mesh filename=meshes/LFinger32_0.10.stl scale=1 1 1; visual mesh filename=meshes/LFinger32.obj scale=1 1 1
- link LFinger33_link: geometry collision mesh filename=meshes/LFinger33_0.10.stl scale=1 1 1; visual mesh filename=meshes/LFinger33.obj scale=1 1 1
- link LShoulderYaw_link: geometry collision mesh filename=meshes/LShoulderYaw_0.10.stl scale=1 1 1; visual mesh filename=meshes/LShoulderYaw_mainskin.obj scale=1 1 1
- link LThigh: geometry collision mesh filename=meshes/LHipPitch_0.10.stl scale=1 1 1; visual mesh filename=meshes/LHipPitch_mainskin.obj scale=1 1 1
- link LTibia: geometry collision mesh filename=meshes/LKneePitch_0.10.stl scale=1 1 1; visual mesh filename=meshes/LKneePitch_mainskin.obj scale=1 1 1
- link l_ankle: geometry collision mesh filename=meshes/LAnkleRoll_0.10.stl scale=1 1 1; visual mesh filename=meshes/LAnkleRoll_mainskin.obj scale=1 1 1
Joints:
- added joint LAnkleRoll_secondaryskin2_joint: type fixed, parent l_ankle, child LAnkleRoll_secondaryskin2, origin xyz=0 0 0 rpy=0 0 0
- added joint LAnkleRoll_secondaryskin_joint: type fixed, parent l_ankle, child LAnkleRoll_secondaryskin, origin xyz=0 0 0 rpy=0 0 0
- added joint LElbowYaw_shell_joint: type fixed, parent LElbow, child LElbowYaw_shell, origin xyz=0 0 0 rpy=0 0 0
- added joint LHipPitch_flexibleskin_joint: type fixed, parent LThigh, child LHipPitch_flexibleskin, origin xyz=0 0 0 rpy=0 0 0
- added joint LHipPitch_secondaryskin_joint: type fixed, parent LThigh, child LHipPitch_secondaryskin, origin xyz=0 0 0 rpy=0 0 0
- added joint LHipPitch_shell_joint: type fixed, parent LThigh, child LHipPitch_shell, origin xyz=0 0 0 rpy=0 0 0
- added joint LKneePitch_secondaryskin2_joint: type fixed, parent LTibia, child LKneePitch_secondaryskin2, origin xyz=0 0 0 rpy=0 0 0
- added joint LKneePitch_secondaryskin3_joint: type fixed, parent LTibia, child LKneePitch_secondaryskin3, origin xyz=0 0 0 rpy=0 0 0
- added joint LKneePitch_secondaryskin_joint: type fixed, parent LTibia, child LKneePitch_secondaryskin, origin xyz=0 0 0 rpy=0 0 0
- added joint LKneePitch_shell_joint: type fixed, parent LTibia, child LKneePitch_shell, origin xyz=0 0 0 rpy=0 0 0
- added joint LShoulderYaw_shell_joint: type fixed, parent LShoulderYaw_link, child LShoulderYaw_shell, origin xyz=0 0 0 rpy=0 0 0

Commit message: Additional batch of converted meshes

File: qibullet/robot_data/romeo_H37/romeo.urdf (robot description, URDF)
Before this commit: robot RomeoH37, 93 links, 92 joints
Links:
- added link RAnkleRoll_secondaryskin, mass 0; visual mesh filename=meshes/RAnkleRoll_secondaryskin.obj scale=1 1 1
- added link RAnkleRoll_secondaryskin2, mass 0; visual mesh filename=meshes/RAnkleRoll_secondaryskin2.obj scale=1 1 1
- link LThumb1_link: geometry collision mesh filename=meshes/LThumb1_0.10.stl scale=1 1 1; visual mesh filename=meshes/LThumb1.obj scale=1 1 1
- link LThumb2_link: geometry collision mesh filename=meshes/LThumb2_0.10.stl scale=1 1 1; visual mesh filename=meshes/LThumb2.obj scale=1 1 1
- link LThumb3_link: geometry collision mesh filename=meshes/LThumb3_0.10.stl scale=1 1 1; visual mesh filename=meshes/LThumb3.obj scale=1 1 1
- link LWristRoll_link: geometry collision mesh filename=meshes/LWristRoll_0.10.stl scale=1 1 1; visual mesh filename=meshes/LWristRoll.obj scale=1 1 1
- link LWristYaw_link: geometry collision mesh filename=meshes/LWristYaw_0.10.stl scale=1 1 1; visual mesh filename=meshes/LWristYaw.obj scale=1 1 1
- link NeckPitch_link: geometry collision mesh filename=meshes/NeckPitch_0.10.stl scale=1 1 1; visual mesh filename=meshes/NeckPitch.obj scale=1 1 1
- link l_wrist: geometry collision mesh filename=meshes/LWristPitch_0.10.stl scale=1 1 1; visual mesh filename=meshes/LWristPitch.obj scale=1 1 1
- link r_ankle: geometry collision mesh filename=meshes/RAnkleRoll_0.10.stl scale=1 1 1; visual mesh filename=meshes/RAnkleRoll_mainskin.obj scale=1 1 1
Joints:
- added joint RAnkleRoll_secondaryskin2_joint: type fixed, parent r_ankle, child RAnkleRoll_secondaryskin2, origin xyz=0 0 0 rpy=0 0 0
- added joint RAnkleRoll_secondaryskin_joint: type fixed, parent r_ankle, child RAnkleRoll_secondaryskin, origin xyz=0 0 0 rpy=0 0 0
