Commit message: Finish converting the meshes

File: qibullet/robot_data/romeo_H37/romeo.urdf (robot description, URDF)
Before this commit: robot RomeoH37, 95 links, 94 joints
Links:
- added link RElbowYaw_shell, mass 0; visual mesh filename=meshes/RElbowYaw_shell.obj scale=1 1 1
- added link RHipPitch_flexibleskin, mass 0; visual mesh filename=meshes/RHipPitch_flexibleskin.obj scale=1 1 1
- added link RHipPitch_secondaryskin, mass 0; visual mesh filename=meshes/RHipPitch_secondaryskin.obj scale=1 1 1
- added link RHipPitch_shell, mass 0; visual mesh filename=meshes/RHipPitch_shell.obj scale=1 1 1
- added link RKneePitch_secondaryskin, mass 0; visual mesh filename=meshes/RKneePitch_secondaryskin.obj scale=1 1 1
- added link RKneePitch_secondaryskin2, mass 0; visual mesh filename=meshes/RKneePitch_secondaryskin2.obj scale=1 1 1
- added link RKneePitch_secondaryskin3, mass 0; visual mesh filename=meshes/RKneePitch_secondaryskin3.obj scale=1 1 1
- added link RKneePitch_shell, mass 0; visual mesh filename=meshes/RKneePitch_shell.obj scale=1 1 1
- added link RShoulderYaw_shell, mass 0; visual mesh filename=meshes/RShoulderYaw_shell.obj scale=1 1 1
- added link TrunkYaw_mainskin, mass 0; visual mesh filename=meshes/TrunkYaw_mainskin.obj scale=1 1 1
- added link TrunkYaw_shell, mass 0; visual mesh filename=meshes/TrunkYaw_shell.obj scale=1 1 1
- added link torso_emergencybutton, mass 0; visual mesh filename=meshes/Torso_emergencybutton.obj scale=1 1 1
- added link torso_flexibleskin, mass 0; visual mesh filename=meshes/Torso_flexibleskin.obj scale=1 1 1
- added link torso_mainskin, mass 0; visual mesh filename=meshes/Torso_mainskin.obj scale=1 1 1
- added link torso_secondaryskin, mass 0; visual mesh filename=meshes/Torso_secondaryskin.obj scale=1 1 1
- added link torso_shell, mass 0; visual mesh filename=meshes/Torso_shell.obj scale=1 1 1
- link RElbow: geometry collision mesh filename=meshes/RElbowYaw_0.10.stl scale=1 1 1; visual mesh filename=meshes/RElbowYaw_mainskin.obj scale=1 1 1
- link REye: geometry collision mesh filename=meshes/REyePitch_0.10.stl scale=1 1 1; visual mesh filename=meshes/REyePitch.obj scale=1 1 1
- link RFinger11_link: geometry collision mesh filename=meshes/RFinger11_0.10.stl scale=1 1 1; visual mesh filename=meshes/RFinger11.obj scale=1 1 1
- link RFinger12_link: geometry collision mesh filename=meshes/RFinger12_0.10.stl scale=1 1 1; visual mesh filename=meshes/RFinger12.obj scale=1 1 1
- link RFinger13_link: geometry collision mesh filename=meshes/RFinger13_0.10.stl scale=1 1 1; visual mesh filename=meshes/RFinger13.obj scale=1 1 1
- link RFinger21_link: geometry collision mesh filename=meshes/RFinger21_0.10.stl scale=1 1 1; visual mesh filename=meshes/RFinger21.obj scale=1 1 1
- link RFinger22_link: geometry collision mesh filename=meshes/RFinger22_0.10.stl scale=1 1 1; visual mesh filename=meshes/RFinger22.obj scale=1 1 1
- link RFinger23_link: geometry collision mesh filename=meshes/RFinger23_0.10.stl scale=1 1 1; visual mesh filename=meshes/RFinger23.obj scale=1 1 1
- link RFinger31_link: geometry collision mesh filename=meshes/RFinger31_0.10.stl scale=1 1 1; visual mesh filename=meshes/RFinger31.obj scale=1 1 1
- link RFinger32_link: geometry collision mesh filename=meshes/RFinger32_0.10.stl scale=1 1 1; visual mesh filename=meshes/RFinger32.obj scale=1 1 1
- link RFinger33_link: geometry collision mesh filename=meshes/RFinger33_0.10.stl scale=1 1 1; visual mesh filename=meshes/RFinger33.obj scale=1 1 1
- link RShoulderYaw_link: geometry collision mesh filename=meshes/RShoulderYaw_0.10.stl scale=1 1 1; visual mesh filename=meshes/RShoulderYaw_mainskin.obj scale=1 1 1
- link RThigh: geometry collision mesh filename=meshes/RHipPitch_0.10.stl scale=1 1 1; visual mesh filename=meshes/RHipPitch_mainskin.obj scale=1 1 1
- link RThumb1_link: geometry collision mesh filename=meshes/RThumb1_0.10.stl scale=1 1 1; visual mesh filename=meshes/RThumb1.obj scale=1 1 1
- link RThumb2_link: geometry collision mesh filename=meshes/RThumb2_0.10.stl scale=1 1 1; visual mesh filename=meshes/RThumb2.obj scale=1 1 1
- link RThumb3_link: geometry collision mesh filename=meshes/RThumb3_0.10.stl scale=1 1 1; visual mesh filename=meshes/RThumb3.obj scale=1 1 1
- link RTibia: geometry collision mesh filename=meshes/RKneePitch_0.10.stl scale=1 1 1; visual mesh filename=meshes/RKneePitch_mainskin.obj scale=1 1 1
- link RWristRoll_link: geometry collision mesh filename=meshes/RWristRoll_0.10.stl scale=1 1 1; visual mesh filename=meshes/RWristRoll.obj scale=1 1 1
- link RWristYaw_link: geometry collision mesh filename=meshes/RWristYaw_0.10.stl scale=1 1 1; visual mesh filename=meshes/RWristYaw.obj scale=1 1 1
- link body: geometry collision mesh filename=meshes/TrunkYaw_0.10.stl scale=1 1 1; visual mesh filename=meshes/TrunkYaw_flexibleskin.obj scale=1 1 1
- link r_wrist: geometry collision mesh filename=meshes/RWristPitch_0.10.stl scale=1 1 1; visual mesh filename=meshes/RWristPitch.obj scale=1 1 1
- link torso: geometry collision mesh filename=meshes/Torso_0.10.stl scale=1 1 1; visual mesh filename=meshes/Torso_logo.obj scale=1 1 1
Joints:
- added joint RElbowYaw_shell_joint: type fixed, parent RElbow, child RElbowYaw_shell, origin xyz=0 0 0 rpy=0 0 0
- added joint RHipPitch_flexibleskin_joint: type fixed, parent RThigh, child RHipPitch_flexibleskin, origin xyz=0 0 0 rpy=0 0 0
- added joint RHipPitch_secondaryskin_joint: type fixed, parent RThigh, child RHipPitch_secondaryskin, origin xyz=0 0 0 rpy=0 0 0
- added joint RHipPitch_shell_joint: type fixed, parent RThigh, child RHipPitch_shell, origin xyz=0 0 0 rpy=0 0 0
- added joint RKneePitch_secondaryskin2_joint: type fixed, parent RTibia, child RKneePitch_secondaryskin2, origin xyz=0 0 0 rpy=0 0 0
- added joint RKneePitch_secondaryskin3_joint: type fixed, parent RTibia, child RKneePitch_secondaryskin3, origin xyz=0 0 0 rpy=0 0 0
- added joint RKneePitch_secondaryskin_joint: type fixed, parent RTibia, child RKneePitch_secondaryskin, origin xyz=0 0 0 rpy=0 0 0
- added joint RKneePitch_shell_joint: type fixed, parent RTibia, child RKneePitch_shell, origin xyz=0 0 0 rpy=0 0 0
- added joint RShoulderYaw_shell_joint: type fixed, parent RShoulderYaw_link, child RShoulderYaw_shell, origin xyz=0 0 0 rpy=0 0 0
- added joint TrunkYaw_mainskin_joint: type fixed, parent body, child TrunkYaw_mainskin, origin xyz=0 0 0 rpy=0 0 0
- added joint TrunkYaw_shell_joint: type fixed, parent body, child TrunkYaw_shell, origin xyz=0 0 0 rpy=0 0 0
- added joint torso_emergencybutton_joint: type fixed, parent torso, child torso_emergencybutton, origin xyz=0 0 0 rpy=0 0 0
- added joint torso_flexibleskin_joint: type fixed, parent torso, child torso_flexibleskin, origin xyz=0 0 0 rpy=0 0 0
- added joint torso_mainskin_joint: type fixed, parent torso, child torso_mainskin, origin xyz=0 0 0 rpy=0 0 0
- added joint torso_secondaryskin_joint: type fixed, parent torso, child torso_secondaryskin, origin xyz=0 0 0 rpy=0 0 0
- added joint torso_shell_joint: type fixed, parent torso, child torso_shell, origin xyz=0 0 0 rpy=0 0 0

Commit message: FInal URDF mass and inertia update

File: qibullet/robot_data/romeo_H37/romeo.urdf (robot description, URDF)
Before this commit: robot RomeoH37, 111 links, 110 joints
Links:
- link CameraDepth_frame: mass None -> 0
- link CameraDepth_optical_frame: mass None -> 0
- link CameraLeftEye_frame: mass None -> 0
- link CameraLeftEye_optical_frame: mass None -> 0
- link CameraLeft_frame: mass None -> 0
- link CameraLeft_optical_frame: mass None -> 0
- link CameraRightEye_frame: mass None -> 0
- link CameraRightEye_optical_frame: mass None -> 0
- link CameraRight_frame: mass None -> 0
- link CameraRight_optical_frame: mass None -> 0
- link ImuHeadAccelerometer_frame: mass None -> 0
- link ImuHeadGyrometer_frame: mass None -> 0
- link ImuTorsoAccelerometer_frame: mass None -> 0
- link ImuTorsoGyrometer_frame: mass None -> 0
- link base_link: mass None -> 0
- link gaze: mass None -> 0
- link l_sole: mass None -> 0
- link r_sole: mass None -> 0

Commit message: Remove balance constraint, add elementary mass to base link

File: qibullet/robot_data/romeo_H37/romeo.urdf (robot description, URDF)
Before this commit: robot RomeoH37, 111 links, 110 joints
Links:
- link base_link: mass 0 -> 0.0000000001

Commit message: Update URDF intertia matrix

File: qibullet/robot_data/romeo_H37/romeo.urdf (robot description, URDF)
Before this commit: robot RomeoH37, 111 links, 110 joints
Links:
- link base_link: mass 0.0000000001 -> 0.00000001
