Commit message: Revisited structure for the whole package

File: qibullet/robot_data/pepper_1.7/pepper.urdf (robot description, URDF)
Before this commit: robot JulietteY20MP, 93 links, 92 joints
Links:
- link Head: geometry collision mesh filename=meshes/HeadPitch_0.10.stl scale=0.1 0.1 0.1; visual mesh filename=meshes/HeadPitch_eyes.obj scale=0.1 0.1 0.1
- link HeadPitch_ears: geometry visual mesh filename=meshes/HeadPitch_ears.obj scale=0.1 0.1 0.1
- link HeadPitch_milky: geometry visual mesh filename=meshes/HeadPitch_milky.obj scale=0.1 0.1 0.1
- link HeadPitch_shiny: geometry visual mesh filename=meshes/HeadPitch_shiny.obj scale=0.1 0.1 0.1
- link Hip: geometry collision mesh filename=meshes/HipRoll_0.10.stl scale=0.1 0.1 0.1; visual mesh filename=meshes/HipRoll.obj scale=0.1 0.1 0.1
- link HipPitch_shiny: geometry visual mesh filename=meshes/HipPitch_shiny.obj scale=0.1 0.1 0.1
- link KneePitch_milky: geometry visual mesh filename=meshes/KneePitch_milky.obj scale=0.1 0.1 0.1
- link LBicep: geometry collision mesh filename=meshes/LShoulderRoll_0.10.stl scale=0.1 0.1 0.1; visual mesh filename=meshes/LShoulderRoll_milky.obj scale=0.1 0.1 0.1
- link LElbow: geometry collision mesh filename=meshes/LElbowYaw_0.10.stl scale=0.1 0.1 0.1; visual mesh filename=meshes/LElbowYaw.obj scale=0.1 0.1 0.1
- link LElbowRoll_milky: geometry visual mesh filename=meshes/LElbowRoll_milky.obj scale=0.1 0.1 0.1
- link LFinger11_link: geometry collision mesh filename=meshes/LFinger11_0.10.stl scale=0.1 0.1 0.1; visual mesh filename=meshes/LFinger11.obj scale=0.1 0.1 0.1
- link LFinger12_link: geometry collision mesh filename=meshes/LFinger12_0.10.stl scale=0.1 0.1 0.1; visual mesh filename=meshes/LFinger12.obj scale=0.1 0.1 0.1
- link LFinger13_link: geometry collision mesh filename=meshes/LFinger13_0.10.stl scale=0.1 0.1 0.1; visual mesh filename=meshes/LFinger13.obj scale=0.1 0.1 0.1
- link LFinger21_link: geometry collision mesh filename=meshes/LFinger21_0.10.stl scale=0.1 0.1 0.1; visual mesh filename=meshes/LFinger21.obj scale=0.1 0.1 0.1
- link LFinger22_link: geometry collision mesh filename=meshes/LFinger22_0.10.stl scale=0.1 0.1 0.1; visual mesh filename=meshes/LFinger22.obj scale=0.1 0.1 0.1
- link LFinger23_link: geometry collision mesh filename=meshes/LFinger23_0.10.stl scale=0.1 0.1 0.1; visual mesh filename=meshes/LFinger23.obj scale=0.1 0.1 0.1
- link LFinger31_link: geometry collision mesh filename=meshes/LFinger31_0.10.stl scale=0.1 0.1 0.1; visual mesh filename=meshes/LFinger31.obj scale=0.1 0.1 0.1
- link LFinger32_link: geometry collision mesh filename=meshes/LFinger32_0.10.stl scale=0.1 0.1 0.1; visual mesh filename=meshes/LFinger32.obj scale=0.1 0.1 0.1
- link LFinger33_link: geometry collision mesh filename=meshes/LFinger33_0.10.stl scale=0.1 0.1 0.1; visual mesh filename=meshes/LFinger33.obj scale=0.1 0.1 0.1
- link LFinger41_link: geometry collision mesh filename=meshes/LFinger41_0.10.stl scale=0.1 0.1 0.1; visual mesh filename=meshes/LFinger41.obj scale=0.1 0.1 0.1
- link LFinger42_link: geometry collision mesh filename=meshes/LFinger42_0.10.stl scale=0.1 0.1 0.1; visual mesh filename=meshes/LFinger42.obj scale=0.1 0.1 0.1
- link LFinger43_link: geometry collision mesh filename=meshes/LFinger43_0.10.stl scale=0.1 0.1 0.1; visual mesh filename=meshes/LFinger43.obj scale=0.1 0.1 0.1
- link LForeArm: geometry collision mesh filename=meshes/LElbowRoll_0.10.stl scale=0.1 0.1 0.1; visual mesh filename=meshes/LElbowRoll_shiny.obj scale=0.1 0.1 0.1
- link LShoulder: geometry collision mesh filename=meshes/LShoulderPitch_0.10.stl scale=0.1 0.1 0.1; visual mesh filename=meshes/LShoulderPitch.obj scale=0.1 0.1 0.1
- link LShoulderRoll_shiny: geometry visual mesh filename=meshes/LShoulderRoll_shiny.obj scale=0.1 0.1 0.1
- link LThumb1_link: geometry collision mesh filename=meshes/LThumb1_0.10.stl scale=0.1 0.1 0.1; visual mesh filename=meshes/LThumb1.obj scale=0.1 0.1 0.1
- link LThumb2_link: geometry collision mesh filename=meshes/LThumb2_0.10.stl scale=0.1 0.1 0.1; visual mesh filename=meshes/LThumb2.obj scale=0.1 0.1 0.1
- link Neck: geometry collision mesh filename=meshes/HeadYaw_0.10.stl scale=0.1 0.1 0.1; visual mesh filename=meshes/HeadYaw.obj scale=0.1 0.1 0.1
- link Pelvis: geometry collision mesh filename=meshes/HipPitch_0.10.stl scale=0.1 0.1 0.1; visual mesh filename=meshes/HipPitch_milky.obj scale=0.1 0.1 0.1
- link RBicep: geometry collision mesh filename=meshes/RShoulderRoll_0.10.stl scale=0.1 0.1 0.1; visual mesh filename=meshes/RShoulderRoll_milky.obj scale=0.1 0.1 0.1
- link RElbow: geometry collision mesh filename=meshes/RElbowYaw_0.10.stl scale=0.1 0.1 0.1; visual mesh filename=meshes/RElbowYaw.obj scale=0.1 0.1 0.1
- link RElbowRoll_milky: geometry visual mesh filename=meshes/RElbowRoll_milky.obj scale=0.1 0.1 0.1
- link RFinger11_link: geometry collision mesh filename=meshes/RFinger11_0.10.stl scale=0.1 0.1 0.1; visual mesh filename=meshes/RFinger11.obj scale=0.1 0.1 0.1
- link RFinger12_link: geometry collision mesh filename=meshes/RFinger12_0.10.stl scale=0.1 0.1 0.1; visual mesh filename=meshes/RFinger12.obj scale=0.1 0.1 0.1
- link RFinger13_link: geometry collision mesh filename=meshes/RFinger13_0.10.stl scale=0.1 0.1 0.1; visual mesh filename=meshes/RFinger13.obj scale=0.1 0.1 0.1
- link RFinger21_link: geometry collision mesh filename=meshes/RFinger21_0.10.stl scale=0.1 0.1 0.1; visual mesh filename=meshes/RFinger21.obj scale=0.1 0.1 0.1
- link RFinger22_link: geometry collision mesh filename=meshes/RFinger22_0.10.stl scale=0.1 0.1 0.1; visual mesh filename=meshes/RFinger22.obj scale=0.1 0.1 0.1
- link RFinger23_link: geometry collision mesh filename=meshes/RFinger23_0.10.stl scale=0.1 0.1 0.1; visual mesh filename=meshes/RFinger23.obj scale=0.1 0.1 0.1
- link RFinger31_link: geometry collision mesh filename=meshes/RFinger31_0.10.stl scale=0.1 0.1 0.1; visual mesh filename=meshes/RFinger31.obj scale=0.1 0.1 0.1
- link RFinger32_link: geometry collision mesh filename=meshes/RFinger32_0.10.stl scale=0.1 0.1 0.1; visual mesh filename=meshes/RFinger32.obj scale=0.1 0.1 0.1
- link RFinger33_link: geometry collision mesh filename=meshes/RFinger33_0.10.stl scale=0.1 0.1 0.1; visual mesh filename=meshes/RFinger33.obj scale=0.1 0.1 0.1
- link RFinger41_link: geometry collision mesh filename=meshes/RFinger41_0.10.stl scale=0.1 0.1 0.1; visual mesh filename=meshes/RFinger41.obj scale=0.1 0.1 0.1
- link RFinger42_link: geometry collision mesh filename=meshes/RFinger42_0.10.stl scale=0.1 0.1 0.1; visual mesh filename=meshes/RFinger42.obj scale=0.1 0.1 0.1
- link RFinger43_link: geometry collision mesh filename=meshes/RFinger43_0.10.stl scale=0.1 0.1 0.1; visual mesh filename=meshes/RFinger43.obj scale=0.1 0.1 0.1
- link RForeArm: geometry collision mesh filename=meshes/RElbowRoll_0.10.stl scale=0.1 0.1 0.1; visual mesh filename=meshes/RElbowRoll_shiny.obj scale=0.1 0.1 0.1
- link RShoulder: geometry collision mesh filename=meshes/RShoulderPitch_0.10.stl scale=0.1 0.1 0.1; visual mesh filename=meshes/RShoulderPitch.obj scale=0.1 0.1 0.1
- link RShoulderRoll_shiny: geometry visual mesh filename=meshes/RShoulderRoll_shiny.obj scale=0.1 0.1 0.1
- link RThumb1_link: geometry collision mesh filename=meshes/RThumb1_0.10.stl scale=0.1 0.1 0.1; visual mesh filename=meshes/RThumb1.obj scale=0.1 0.1 0.1
- link RThumb2_link: geometry collision mesh filename=meshes/RThumb2_0.10.stl scale=0.1 0.1 0.1; visual mesh filename=meshes/RThumb2.obj scale=0.1 0.1 0.1
- link Tibia: geometry collision mesh filename=meshes/KneePitch_0.10.stl scale=0.1 0.1 0.1; visual mesh filename=meshes/KneePitch_shiny.obj scale=0.1 0.1 0.1
- link Torso_shiny: geometry visual mesh filename=meshes/Torso_shiny.obj scale=0.1 0.1 0.1
- link Torso_transparent: geometry visual mesh filename=meshes/Torso_transparent.obj scale=0.1 0.1 0.1
- link WheelB_link: geometry collision mesh filename=meshes/WheelB_0.10.stl scale=0.1 0.1 0.1; visual mesh filename=meshes/WheelB.obj scale=0.1 0.1 0.1
- link WheelFL_link: geometry collision mesh filename=meshes/WheelFL_0.10.stl scale=0.1 0.1 0.1; visual mesh filename=meshes/WheelFL.obj scale=0.1 0.1 0.1
- link WheelFR_link: geometry collision mesh filename=meshes/WheelFR_0.10.stl scale=0.1 0.1 0.1; visual mesh filename=meshes/WheelFR.obj scale=0.1 0.1 0.1
- link l_wrist: geometry collision mesh filename=meshes/LWristYaw_0.10.stl scale=0.1 0.1 0.1; visual mesh filename=meshes/LWristYaw.obj scale=0.1 0.1 0.1
- link r_wrist: geometry collision mesh filename=meshes/RWristYaw_0.10.stl scale=0.1 0.1 0.1; visual mesh filename=meshes/RWristYaw.obj scale=0.1 0.1 0.1
- link torso: geometry collision mesh filename=meshes/Torso_0.10.stl scale=0.1 0.1 0.1; visual mesh filename=meshes/Torso_milky.obj scale=0.1 0.1 0.1

Commit message: Update all finger from continuous to revolute joints

File: qibullet/robot_data/pepper_1.7/pepper.urdf (robot description, URDF)
Before this commit: robot JulietteY20MP, 93 links, 92 joints
Joints:
- joint LFinger11: type continuous -> revolute
- joint LFinger12: type continuous -> revolute
- joint LFinger13: type continuous -> revolute
- joint LFinger21: type continuous -> revolute
- joint LFinger22: type continuous -> revolute
- joint LFinger23: type continuous -> revolute
- joint LFinger31: type continuous -> revolute
- joint LFinger32: type continuous -> revolute
- joint LFinger33: type continuous -> revolute
- joint LFinger41: type continuous -> revolute
- joint LFinger42: type continuous -> revolute
- joint LFinger43: type continuous -> revolute
- joint LThumb1: type continuous -> revolute
- joint LThumb2: type continuous -> revolute
- joint RFinger11: type continuous -> revolute
- joint RFinger12: type continuous -> revolute
- joint RFinger13: type continuous -> revolute
- joint RFinger21: type continuous -> revolute
- joint RFinger22: type continuous -> revolute
- joint RFinger23: type continuous -> revolute
- joint RFinger31: type continuous -> revolute
- joint RFinger32: type continuous -> revolute
- joint RFinger33: type continuous -> revolute
- joint RFinger41: type continuous -> revolute
- joint RFinger42: type continuous -> revolute
- joint RFinger43: type continuous -> revolute
- joint RThumb1: type continuous -> revolute
- joint RThumb2: type continuous -> revolute

Commit message: Add the necessary masses and inertial missing informations

File: qibullet/robot_data/pepper_1.7/pepper.urdf (robot description, URDF)
Before this commit: robot JulietteY20MP, 93 links, 92 joints
Links:
- link BumperB_frame: mass None -> 0
- link BumperFL_frame: mass None -> 0
- link BumperFR_frame: mass None -> 0
- link CameraBottom_frame: mass None -> 0
- link CameraBottom_optical_frame: mass None -> 0
- link CameraDepth_frame: mass None -> 0
- link CameraDepth_optical_frame: mass None -> 0
- link CameraTop_frame: mass None -> 0
- link CameraTop_optical_frame: mass None -> 0
- link ChestButton_frame: mass None -> 0
- link HeadPitch_ears: mass None -> 0
- link HeadPitch_milky: mass None -> 0
- link HeadPitch_shiny: mass None -> 0
- link HeadTouchFront_frame: mass None -> 0
- link HeadTouchMiddle_frame: mass None -> 0
- link HeadTouchRear_frame: mass None -> 0
- link HipPitch_shiny: mass None -> 0
- link ImuBaseAccelerometer_frame: mass None -> 0
- link ImuTorsoAccelerometer_frame: mass None -> 0
- link ImuTorsoGyrometer_frame: mass None -> 0
- link KneePitch_milky: mass None -> 0
- link LElbowRoll_milky: mass None -> 0
- link LHandTouchBack_frame: mass None -> 0
- link LShoulderRoll_shiny: mass None -> 0
- link LSpeaker_frame: mass None -> 0
- link RElbowRoll_milky: mass None -> 0
- link RHandTouchBack_frame: mass None -> 0
- link RShoulderRoll_shiny: mass None -> 0
- link RSpeaker_frame: mass None -> 0
- link ShovelLaser_frame: mass None -> 0
- link SonarBack_frame: mass None -> 0
- link SonarFront_frame: mass None -> 0
- link SurroundingFrontLaser_device_frame: mass None -> 0
- link SurroundingFrontLaser_frame: mass None -> 0
- link SurroundingLeftLaser_device_frame: mass None -> 0
- link SurroundingLeftLaser_frame: mass None -> 0
- link SurroundingRightLaser_device_frame: mass None -> 0
- link SurroundingRightLaser_frame: mass None -> 0
- link Tablet_frame: mass None -> 0
- link Torso_shiny: mass None -> 0
- link Torso_transparent: mass None -> 0
- link VerticalLeftLaser_frame: mass None -> 0
- link VerticalRightLaser_frame: mass None -> 0
- link base_footprint: mass None -> 0

Commit message: Update Pepper's hand collision files

File: qibullet/robot_data/pepper_1.7/pepper.urdf (robot description, URDF)
Before this commit: robot JulietteY20MP, 93 links, 92 joints
Links:
- link LFinger11_link: geometry collision mesh filename=meshes/LFinger11.dae scale=0.1 0.1 0.1; visual mesh filename=meshes/LFinger11.obj scale=0.1 0.1 0.1
- link LFinger12_link: geometry collision mesh filename=meshes/LFinger12.dae scale=0.1 0.1 0.1; visual mesh filename=meshes/LFinger12.obj scale=0.1 0.1 0.1
- link LFinger13_link: geometry collision mesh filename=meshes/LFinger13.dae scale=0.1 0.1 0.1; visual mesh filename=meshes/LFinger13.obj scale=0.1 0.1 0.1
- link LFinger21_link: geometry collision mesh filename=meshes/LFinger21.dae scale=0.1 0.1 0.1; visual mesh filename=meshes/LFinger21.obj scale=0.1 0.1 0.1
- link LFinger22_link: geometry collision mesh filename=meshes/LFinger22.dae scale=0.1 0.1 0.1; visual mesh filename=meshes/LFinger22.obj scale=0.1 0.1 0.1
- link LFinger23_link: geometry collision mesh filename=meshes/LFinger23.dae scale=0.1 0.1 0.1; visual mesh filename=meshes/LFinger23.obj scale=0.1 0.1 0.1
- link LFinger31_link: geometry collision mesh filename=meshes/LFinger31.dae scale=0.1 0.1 0.1; visual mesh filename=meshes/LFinger31.obj scale=0.1 0.1 0.1
- link LFinger32_link: geometry collision mesh filename=meshes/LFinger32.dae scale=0.1 0.1 0.1; visual mesh filename=meshes/LFinger32.obj scale=0.1 0.1 0.1
- link LFinger33_link: geometry collision mesh filename=meshes/LFinger33.dae scale=0.1 0.1 0.1; visual mesh filename=meshes/LFinger33.obj scale=0.1 0.1 0.1
- link LFinger41_link: geometry collision mesh filename=meshes/LFinger41.dae scale=0.1 0.1 0.1; visual mesh filename=meshes/LFinger41.obj scale=0.1 0.1 0.1
- link LFinger42_link: geometry collision mesh filename=meshes/LFinger42.dae scale=0.1 0.1 0.1; visual mesh filename=meshes/LFinger42.obj scale=0.1 0.1 0.1
- link LFinger43_link: geometry collision mesh filename=meshes/LFinger43.dae scale=0.1 0.1 0.1; visual mesh filename=meshes/LFinger43.obj scale=0.1 0.1 0.1
- link LThumb1_link: geometry collision mesh filename=meshes/LThumb1.dae scale=0.1 0.1 0.1; visual mesh filename=meshes/LThumb1.obj scale=0.1 0.1 0.1
- link LThumb2_link: geometry collision mesh filename=meshes/LThumb2.dae scale=0.1 0.1 0.1; visual mesh filename=meshes/LThumb2.obj scale=0.1 0.1 0.1
- link RFinger11_link: geometry collision mesh filename=meshes/RFinger11.dae scale=0.1 0.1 0.1; visual mesh filename=meshes/RFinger11.obj scale=0.1 0.1 0.1
- link RFinger12_link: geometry collision mesh filename=meshes/RFinger12.dae scale=0.1 0.1 0.1; visual mesh filename=meshes/RFinger12.obj scale=0.1 0.1 0.1
- link RFinger13_link: geometry collision mesh filename=meshes/RFinger13.dae scale=0.1 0.1 0.1; visual mesh filename=meshes/RFinger13.obj scale=0.1 0.1 0.1
- link RFinger21_link: geometry collision mesh filename=meshes/RFinger21.dae scale=0.1 0.1 0.1; visual mesh filename=meshes/RFinger21.obj scale=0.1 0.1 0.1
- link RFinger22_link: geometry collision mesh filename=meshes/RFinger22.dae scale=0.1 0.1 0.1; visual mesh filename=meshes/RFinger22.obj scale=0.1 0.1 0.1
- link RFinger23_link: geometry collision mesh filename=meshes/RFinger23.dae scale=0.1 0.1 0.1; visual mesh filename=meshes/RFinger23.obj scale=0.1 0.1 0.1
- link RFinger31_link: geometry collision mesh filename=meshes/RFinger31.dae scale=0.1 0.1 0.1; visual mesh filename=meshes/RFinger31.obj scale=0.1 0.1 0.1
- link RFinger32_link: geometry collision mesh filename=meshes/RFinger32.dae scale=0.1 0.1 0.1; visual mesh filename=meshes/RFinger32.obj scale=0.1 0.1 0.1
- link RFinger33_link: geometry collision mesh filename=meshes/RFinger33.dae scale=0.1 0.1 0.1; visual mesh filename=meshes/RFinger33.obj scale=0.1 0.1 0.1
- link RFinger41_link: geometry collision mesh filename=meshes/RFinger41.dae scale=0.1 0.1 0.1; visual mesh filename=meshes/RFinger41.obj scale=0.1 0.1 0.1
- link RFinger42_link: geometry collision mesh filename=meshes/RFinger42.dae scale=0.1 0.1 0.1; visual mesh filename=meshes/RFinger42.obj scale=0.1 0.1 0.1
- link RFinger43_link: geometry collision mesh filename=meshes/RFinger43.dae scale=0.1 0.1 0.1; visual mesh filename=meshes/RFinger43.obj scale=0.1 0.1 0.1
- link RThumb1_link: geometry collision mesh filename=meshes/RThumb1.dae scale=0.1 0.1 0.1; visual mesh filename=meshes/RThumb1.obj scale=0.1 0.1 0.1
- link RThumb2_link: geometry collision mesh filename=meshes/RThumb2.dae scale=0.1 0.1 0.1; visual mesh filename=meshes/RThumb2.obj scale=0.1 0.1 0.1
- link l_wrist: geometry collision mesh filename=meshes/LWristYaw.dae scale=0.1 0.1 0.1; visual mesh filename=meshes/LWristYaw.obj scale=0.1 0.1 0.1
- link r_wrist: geometry collision mesh filename=meshes/RWristYaw.dae scale=0.1 0.1 0.1; visual mesh filename=meshes/RWristYaw.obj scale=0.1 0.1 0.1

Commit message: Correct HipRoll rotation

File: qibullet/robot_data/pepper_1.7/pepper.urdf (robot description, URDF)
Before this commit: robot JulietteY20MP, 93 links, 92 joints
Links:
- added link HipOffset
Joints:
- added joint HipOffset_fixed: type fixed, parent HipOffset, child torso, origin xyz=0 0 0.139 rpy=0 0 0
- joint HipRoll: child torso -> HipOffset; origin xyz=-2e-05 0 0.218 rpy=0 0 0 -> xyz=-2e-05 0 0.079 rpy=0 0 0

Commit message: Update the pepper urdf to have a better rotation of the hip

File: qibullet/robot_data/pepper_1.7/pepper.urdf (robot description, URDF)
Before this commit: robot JulietteY20MP, 94 links, 93 joints
Links:
- link HipOffset: mass None -> 0

Commit message: No need for a fixed joint to have a correct hip roll rotation

File: qibullet/robot_data/pepper_1.7/pepper.urdf (robot description, URDF)
Before this commit: robot JulietteY20MP, 94 links, 93 joints
Links:
- removed link HipOffset
Joints:
- removed joint HipOffset_fixed
- joint Accelerometer_sensor_fixedjoint: origin xyz=0.00239 -0.03575 0.00626 rpy=0 0 0 -> xyz=0.00239 -0.03575 0.14526 rpy=0 0 0
- joint ChestBoard/Button_sensor_fixedjoint: origin xyz=0.049871 0.001588 0.055163 rpy=0 0 0 -> xyz=0.049871 0.001588 0.194163 rpy=0 0 0
- joint Gyrometer_sensor_fixedjoint: origin xyz=0.00204 -0.03491 -0.00959 rpy=0 0 0 -> xyz=0.00204 -0.03491 0.12941 rpy=0 0 0
- joint HeadYaw: origin xyz=-0.038 0 0.1699 rpy=0 0 0 -> xyz=-0.038 0 0.3089 rpy=0 0 0
- joint HipRoll: child HipOffset -> torso
- joint LShoulderPitch: origin xyz=-0.057 0.14974 0.08682 rpy=0 0 0 -> xyz=-0.057 0.14974 0.22582 rpy=0 0 0
- joint RShoulderPitch: origin xyz=-0.057 -0.14974 0.08682 rpy=0 0 0 -> xyz=-0.057 -0.14974 0.22582 rpy=0 0 0
- joint Tablet_sensor_fixedjoint: origin xyz=0.0839249 0 0.06251 rpy=0 -0.523599 0 -> xyz=0.0839249 0 0.20151 rpy=0 -0.523599 0
- joint Torso_shiny_joint: origin xyz=0 0 0 rpy=0 0 0 -> xyz=0 0 0.0695 rpy=0 0 0
- joint Torso_transparent_joint: origin xyz=0 0 0 rpy=0 0 0 -> xyz=0 0 0.0695 rpy=0 0 0

Commit message: Add base link in Pepper URDF for more consistency with the ROS stack

File: qibullet/robot_data/pepper_1.7/pepper.urdf (robot description, URDF)
Before this commit: robot JulietteY20MP, 93 links, 92 joints
Links:
- added link base_link, mass 0
Joints:
- added joint base_link_joint: type fixed, parent base_link, child base_footprint, origin xyz=0 0 0 rpy=0 0 0

Commit message: reoriente thumb R/L Signed-off-by: mcaniot <mcaniot@aldebaran.com>

File: qibullet/robot_data/pepper_1.7/pepper.urdf (robot description, URDF)
Before this commit: robot JulietteY20MP, 94 links, 93 joints
Joints:
- joint LThumb1: origin xyz=0.0482 -0.0357 -0.0199 rpy=-1.95836 0.60626 0.533978 -> xyz=0.0482 -0.0357 -0.0199 rpy=-2.55836 0.80626 0.533978
- joint RThumb1: origin xyz=0.0482 0.0357 -0.0199 rpy=-1.18323 0.60626 -0.533978 -> xyz=0.0482 0.0357 -0.0199 rpy=-0.58323 0.80626 -0.533978

Commit message: Update the Pepper URDF, the gripper frames are fixed in the wrist frames, the hand frames are revolute

File: qibullet/robot_data/pepper_1.7/pepper.urdf (robot description, URDF)
Before this commit: robot JulietteY20MP, 94 links, 93 joints
Links:
- added link l_hand, mass 2e-03
- added link r_hand, mass 2e-03
Joints:
- added joint LGripper: type fixed, parent l_wrist, child l_gripper, origin xyz=0.07 0.0 -0.01802319018 rpy=-2.355 0.0 -1.57, axis 0 0 0
- added joint RGripper: type fixed, parent r_wrist, child r_gripper, origin xyz=0.07 0.0 -0.01802319018 rpy=2.355 0 1.57, axis 0 0 0
- joint LHand: child l_gripper -> l_hand
- joint RHand: child r_gripper -> r_hand
