Commit message: Update Pepper URDF for the new meshes

File: qibullet/robot_data/pepper.urdf (robot description, URDF)
Before this commit: robot JulietteY20MP, 96 links, 95 joints
Links:
- removed link HeadPitch_ears
- removed link HeadPitch_milky
- removed link HeadPitch_shiny
- removed link HipPitch_shiny
- removed link KneePitch_milky
- removed link LElbowRoll_milky
- removed link LShoulderRoll_shiny
- removed link RElbowRoll_milky
- removed link RShoulderRoll_shiny
- removed link Torso_shiny
- removed link Torso_transparent
- added link HeadPitch_1, mass 0; visual mesh filename=meshes/pepper/HeadPitch_1.obj scale=1 1 1
- added link HeadPitch_2, mass 0; visual mesh filename=meshes/pepper/HeadPitch_2.obj scale=1 1 1
- added link HeadPitch_3, mass 0; visual mesh filename=meshes/pepper/HeadPitch_3.obj scale=1 1 1
- added link HeadPitch_4, mass 0; visual mesh filename=meshes/pepper/HeadPitch_4.obj scale=1 1 1
- added link HipPitch_1, mass 0; visual mesh filename=meshes/pepper/HipPitch_1.obj scale=1 1 1
- added link KneePitch_1, mass 0; visual mesh filename=meshes/pepper/KneePitch_1.obj scale=1 1 1
- added link LElbowRoll_1, mass 0; visual mesh filename=meshes/pepper/LElbowRoll_1.obj scale=1 1 1
- added link LShoulderRoll_1, mass 0; visual mesh filename=meshes/pepper/LShoulderRoll_1.obj scale=1 1 1
- added link RElbowRoll_1, mass 0; visual mesh filename=meshes/pepper/RElbowRoll_1.obj scale=1 1 1
- added link RShoulderRoll_1, mass 0; visual mesh filename=meshes/pepper/RShoulderRoll_1.obj scale=1 1 1
- added link Torso_1, mass 0; visual mesh filename=meshes/pepper/Torso_1.obj scale=1 1 1
- added link Torso_2, mass 0; visual mesh filename=meshes/pepper/Torso_2.obj scale=1 1 1
- added link Torso_3, mass 0; visual mesh filename=meshes/pepper/Torso_3.obj scale=1 1 1
- added link Torso_4, mass 0; visual mesh filename=meshes/pepper/Torso_4.obj scale=1 1 1
- link Head: geometry collision mesh filename=meshes/pepper/HeadPitch_0.10.stl scale=1 1 1; visual mesh filename=meshes/pepper/HeadPitch_0.obj scale=1 1 1
- link Hip: geometry collision mesh filename=meshes/pepper/HipRoll_0.10.stl scale=1 1 1; visual mesh filename=meshes/pepper/HipRoll.obj scale=1 1 1
- link LBicep: geometry collision mesh filename=meshes/pepper/LShoulderRoll_0.10.stl scale=1 1 1; visual mesh filename=meshes/pepper/LShoulderRoll_0.obj scale=1 1 1
- link LElbow: geometry collision mesh filename=meshes/pepper/LElbowYaw_0.10.stl scale=1 1 1; visual mesh filename=meshes/pepper/LElbowYaw.obj scale=1 1 1
- link LFinger11_link: geometry collision mesh filename=meshes/pepper/Phalax.obj scale=1 1 1; visual mesh filename=meshes/pepper/Phalax.obj scale=1 1 1
- link LFinger12_link: geometry collision mesh filename=meshes/pepper/Phalax.obj scale=1 1 1; visual mesh filename=meshes/pepper/Phalax.obj scale=1 1 1
- link LFinger13_link: geometry collision mesh filename=meshes/pepper/PhalaxEnd.obj scale=1 1 1; visual mesh filename=meshes/pepper/PhalaxEnd.obj scale=1 1 1
- link LFinger21_link: geometry collision mesh filename=meshes/pepper/Phalax.obj scale=1 1 1; visual mesh filename=meshes/pepper/Phalax.obj scale=1 1 1
- link LFinger22_link: geometry collision mesh filename=meshes/pepper/Phalax.obj scale=1 1 1; visual mesh filename=meshes/pepper/Phalax.obj scale=1 1 1
- link LFinger23_link: geometry collision mesh filename=meshes/pepper/PhalaxEnd.obj scale=1 1 1; visual mesh filename=meshes/pepper/PhalaxEnd.obj scale=1 1 1
- link LFinger31_link: geometry collision mesh filename=meshes/pepper/Phalax.obj scale=1 1 1; visual mesh filename=meshes/pepper/Phalax.obj scale=1 1 1
- link LFinger32_link: geometry collision mesh filename=meshes/pepper/Phalax.obj scale=1 1 1; visual mesh filename=meshes/pepper/Phalax.obj scale=1 1 1
- link LFinger33_link: geometry collision mesh filename=meshes/pepper/PhalaxEnd.obj scale=1 1 1; visual mesh filename=meshes/pepper/PhalaxEnd.obj scale=1 1 1
- link LFinger41_link: geometry collision mesh filename=meshes/pepper/Phalax.obj scale=1 1 1; visual mesh filename=meshes/pepper/Phalax.obj scale=1 1 1
- link LFinger42_link: geometry collision mesh filename=meshes/pepper/Phalax.obj scale=1 1 1; visual mesh filename=meshes/pepper/Phalax.obj scale=1 1 1
- link LFinger43_link: geometry collision mesh filename=meshes/pepper/PhalaxEnd.obj scale=1 1 1; visual mesh filename=meshes/pepper/PhalaxEnd.obj scale=1 1 1
- link LForeArm: geometry collision mesh filename=meshes/pepper/LElbowRoll_0.10.stl scale=1 1 1; visual mesh filename=meshes/pepper/LElbowRoll_0.obj scale=1 1 1
- link LShoulder: geometry collision mesh filename=meshes/pepper/LShoulderPitch_0.10.stl scale=1 1 1; visual mesh filename=meshes/pepper/LShoulderPitch.obj scale=1 1 1
- link LThumb1_link: geometry collision mesh filename=meshes/pepper/Phalax.obj scale=1 1 1; visual mesh filename=meshes/pepper/Phalax.obj scale=1 1 1
- link LThumb2_link: geometry collision mesh filename=meshes/pepper/PhalaxEnd.obj scale=1 1 1; visual mesh filename=meshes/pepper/PhalaxEnd.obj scale=1 1 1
- link Neck: geometry collision mesh filename=meshes/pepper/HeadYaw_0.10.stl scale=1 1 1; visual mesh filename=meshes/pepper/HeadYaw.obj scale=1 1 1
- link Pelvis: geometry collision mesh filename=meshes/pepper/HipPitch_0.10.stl scale=1 1 1; visual mesh filename=meshes/pepper/HipPitch_0.obj scale=1 1 1
- link RBicep: geometry collision mesh filename=meshes/pepper/RShoulderRoll_0.10.stl scale=1 1 1; visual mesh filename=meshes/pepper/RShoulderRoll_0.obj scale=1 1 1
- link RElbow: geometry collision mesh filename=meshes/pepper/RElbowYaw_0.10.stl scale=1 1 1; visual mesh filename=meshes/pepper/RElbowYaw.obj scale=1 1 1
- link RFinger11_link: geometry collision mesh filename=meshes/pepper/Phalax.obj scale=1 1 1; visual mesh filename=meshes/pepper/Phalax.obj scale=1 1 1
- link RFinger12_link: geometry collision mesh filename=meshes/pepper/Phalax.obj scale=1 1 1; visual mesh filename=meshes/pepper/Phalax.obj scale=1 1 1
- link RFinger13_link: geometry collision mesh filename=meshes/pepper/PhalaxEnd.obj scale=1 1 1; visual mesh filename=meshes/pepper/PhalaxEnd.obj scale=1 1 1
- link RFinger21_link: geometry collision mesh filename=meshes/pepper/Phalax.obj scale=1 1 1; visual mesh filename=meshes/pepper/Phalax.obj scale=1 1 1
- link RFinger22_link: geometry collision mesh filename=meshes/pepper/Phalax.obj scale=1 1 1; visual mesh filename=meshes/pepper/Phalax.obj scale=1 1 1
- link RFinger23_link: geometry collision mesh filename=meshes/pepper/PhalaxEnd.obj scale=1 1 1; visual mesh filename=meshes/pepper/PhalaxEnd.obj scale=1 1 1
- link RFinger31_link: geometry collision mesh filename=meshes/pepper/Phalax.obj scale=1 1 1; visual mesh filename=meshes/pepper/Phalax.obj scale=1 1 1
- link RFinger32_link: geometry collision mesh filename=meshes/pepper/Phalax.obj scale=1 1 1; visual mesh filename=meshes/pepper/Phalax.obj scale=1 1 1
- link RFinger33_link: geometry collision mesh filename=meshes/pepper/PhalaxEnd.obj scale=1 1 1; visual mesh filename=meshes/pepper/PhalaxEnd.obj scale=1 1 1
- link RFinger41_link: geometry collision mesh filename=meshes/pepper/Phalax.obj scale=1 1 1; visual mesh filename=meshes/pepper/Phalax.obj scale=1 1 1
- link RFinger42_link: geometry collision mesh filename=meshes/pepper/Phalax.obj scale=1 1 1; visual mesh filename=meshes/pepper/Phalax.obj scale=1 1 1
- link RFinger43_link: geometry collision mesh filename=meshes/pepper/PhalaxEnd.obj scale=1 1 1; visual mesh filename=meshes/pepper/PhalaxEnd.obj scale=1 1 1
- link RForeArm: geometry collision mesh filename=meshes/pepper/RElbowRoll_0.10.stl scale=1 1 1; visual mesh filename=meshes/pepper/RElbowRoll_0.obj scale=1 1 1
- link RShoulder: geometry collision mesh filename=meshes/pepper/RShoulderPitch_0.10.stl scale=1 1 1; visual mesh filename=meshes/pepper/RShoulderPitch.obj scale=1 1 1
- link RThumb1_link: geometry collision mesh filename=meshes/pepper/Phalax.obj scale=1 1 1; visual mesh filename=meshes/pepper/Phalax.obj scale=1 1 1
- link RThumb2_link: geometry collision mesh filename=meshes/pepper/PhalaxEnd.obj scale=1 1 1; visual mesh filename=meshes/pepper/PhalaxEnd.obj scale=1 1 1
- link Tibia: geometry collision mesh filename=meshes/pepper/KneePitch_0.10.stl scale=1 1 1; visual mesh filename=meshes/pepper/KneePitch_0.obj scale=1 1 1
- link WheelB_link: geometry collision mesh filename=meshes/pepper/Wheel_0.10.stl scale=1 1 1; visual mesh filename=meshes/pepper/Wheel.obj scale=1 1 1
- link WheelFL_link: geometry collision mesh filename=meshes/pepper/Wheel_0.10.stl scale=1 1 1; visual mesh filename=meshes/pepper/Wheel.obj scale=1 1 1
- link WheelFR_link: geometry collision mesh filename=meshes/pepper/Wheel_0.10.stl scale=1 1 1; visual mesh filename=meshes/pepper/Wheel.obj scale=1 1 1
- link l_wrist: geometry collision mesh filename=meshes/pepper/LWristYaw_vhacd.obj scale=1 1 1; visual mesh filename=meshes/pepper/LWristYaw.obj scale=1 1 1
- link r_wrist: geometry collision mesh filename=meshes/pepper/RWristYaw_vhacd.obj scale=1 1 1; visual mesh filename=meshes/pepper/RWristYaw.obj scale=1 1 1
- link torso: geometry collision mesh filename=meshes/pepper/Torso_0.10.stl scale=1 1 1; visual mesh filename=meshes/pepper/Torso_0.obj scale=1 1 1
Joints:
- removed joint HeadPitch_ears_joint
- removed joint HeadPitch_milky_joint
- removed joint HeadPitch_shiny_joint
- removed joint HipPitch_shiny_joint
- removed joint KneePitch_milky_joint
- removed joint LElbowRoll_milky_joint
- removed joint LShoulderRoll_shiny_joint
- removed joint RElbowRoll_milky_joint
- removed joint RShoulderRoll_shiny_joint
- removed joint Torso_shiny_joint
- removed joint Torso_transparent_joint
- added joint HeadPitch_1_joint: type fixed, parent Head, child HeadPitch_1, origin xyz=0 0 0 rpy=0 0 0
- added joint HeadPitch_2_joint: type fixed, parent Head, child HeadPitch_2, origin xyz=0 0 0 rpy=0 0 0
- added joint HeadPitch_3_joint: type fixed, parent Head, child HeadPitch_3, origin xyz=0 0 0 rpy=0 0 0
- added joint HeadPitch_4_joint: type fixed, parent Head, child HeadPitch_4, origin xyz=0 0 0 rpy=0 0 0
- added joint HipPitch_1_joint: type fixed, parent Pelvis, child HipPitch_1, origin xyz=0 0 0 rpy=0 0 0
- added joint KneePitch_1_joint: type fixed, parent Tibia, child KneePitch_1, origin xyz=0 0 0 rpy=0 0 0
- added joint LElbowRoll_1_joint: type fixed, parent LForeArm, child LElbowRoll_1, origin xyz=0 0 0 rpy=0 0 0
- added joint LShoulderRoll_1_joint: type fixed, parent LBicep, child LShoulderRoll_1, origin xyz=0 0 0 rpy=0 0 0
- added joint RElbowRoll_1_joint: type fixed, parent RForeArm, child RElbowRoll_1, origin xyz=0 0 0 rpy=0 0 0
- added joint RShoulderRoll_1_joint: type fixed, parent RBicep, child RShoulderRoll_1, origin xyz=0 0 0 rpy=0 0 0
- added joint Torso_1_joint: type fixed, parent torso, child Torso_1, origin xyz=0 0 0.0695 rpy=0 0 0
- added joint Torso_2_joint: type fixed, parent torso, child Torso_2, origin xyz=0 0 0.0695 rpy=0 0 0
- added joint Torso_3_joint: type fixed, parent torso, child Torso_3, origin xyz=0 0 0.0695 rpy=0 0 0
- added joint Torso_4_joint: type fixed, parent torso, child Torso_4, origin xyz=0 0 0.0695 rpy=0 0 0
